File: Schematics/SDC/Precharge/updatedPrecharge.kicad_sch (KiCad schematic)
At the start: 14 parts, among them J1 Conn_01x06, Q1 VN3205N3-G, Q2 VP3203N3-G, Q4 VP3203N3-G, U1 LM358DR2G

Commit message: TSAL
Other:
- moved on the sheet: C1, D1, D2, D3, J1, Q1, Q2, Q4, R3, U1
