File: Schematics/VIL/voltage_indicator.kicad_sch (KiCad schematic)
At the start: 10 parts, among them Q1 VN2460, Q2 UJ3N120035K3S

Commit message: VIL edit
Other:
- moved on the sheet: D2, D3, F1, Molex1, Molex2, Q1, Q2, R1, R2, R3

Commit message: edits
Changed lines of the file:
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@@
   (symbol (lib_id "Device:R") (at 124.46 64.77 0) (unit 1)
     (in_bom yes) (on_board yes) (dnp no) (fields_autoplaced)
-    (property "Reference" "R3" (at 126.365 63.5 0)
+    (property "Reference" "R3" (at 127 64.135 0)
       (effects (font (size 1.27 1.27)) (justify left))
     )
-    (property "Value" "RK73G2BTTD1004C" (at 126.365 66.04 0)
+    (property "Value" "RK73G2BTTD1004C" (at 127 66.675 0)
       (effects (font (size 1.27 1.27)) (justify left))
     )

Commit message: fixed up boards
Parts:
- R3: value RK73G2BTTD1004C -> PR02000201004FA100; footprint Resistor_SMD:RESC3116X65N -> Resistor_THT:R_Axial_DIN0207_L6.3mm_D2.5mm_P7.62mm_Horizontal
Changed lines of the file:
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@@
   (junction (at 107.95 77.47) (diameter 0) (color 0 0 0 0)
   )
+  (wire (pts (xy 82.55 26.035) (xy 96.52 26.035))
+    (stroke (width 0) (type default))
+  )
+  (wire (pts (xy 96.52 41.91) (xy 96.52 46.355))
+    (stroke (width 0) (type default))
+  )
+  (wire (pts (xy 96.52 90.17) (xy 62.23 90.17))
+    (stroke (width 0) (type default))
+  )
+  (wire (pts (xy 62.23 36.83) (xy 88.9 36.83))
+    (stroke (width 0) (type default))
+  )
+  (wire (pts (xy 107.95 90.17) (xy 124.46 90.17))
+    (stroke (width 0) (type default))
+  )
+  (wire (pts (xy 62.23 36.83) (xy 62.23 28.575))
+    (stroke (width 0) (type default))
+  )
+  (wire (pts (xy 124.46 77.47) (xy 124.46 68.58))
+    (stroke (width 0) (type default))
+  )
+  (wire (pts (xy 107.95 77.47) (xy 107.95 80.01))
+    (stroke (width 0) (type default))
+  )
+  (wire (pts (xy 124.46 90.17) (xy 124.46 87.63))
+    (stroke (width 0) (type default))
+  )
+  (wire (pts (xy 124.46 26.035) (xy 96.52 26.035))
+    (stroke (width 0) (type default))
+  )
+  (wire (pts (xy 107.95 77.47) (xy 124.46 77.47))
+    (stroke (width 0) (type default))
+  )
+  (wire (pts (xy 96.52 26.035) (xy 96.52 31.75))
+    (stroke (width 0) (type default))
+  )
+  (wire (pts (xy 62.23 26.035) (xy 74.93 26.035))
+    (stroke (width 0) (type default))
+  )
   (wire (pts (xy 124.46 49.53) (xy 124.46 60.96))
-    (stroke (width 0) (type default))
-  )
-  (wire (pts (xy 82.55 26.035) (xy 96.52 26.035))
-    (stroke (width 0) (type default))
-  )
-  (wire (pts (xy 96.52 41.91) (xy 96.52 46.355))
-    (stroke (width 0) (type default))
-  )
-  (wire (pts (xy 96.52 90.17) (xy 62.23 90.17))
-    (stroke (width 0) (type default))
-  )
-  (wire (pts (xy 62.23 36.83) (xy 88.9 36.83))
-    (stroke (width 0) (type default))
-  )
-  (wire (pts (xy 107.95 90.17) (xy 124.46 90.17))
-    (stroke (width 0) (type default))
-  )
-  (wire (pts (xy 62.23 36.83) (xy 62.23 28.575))
-    (stroke (width 0) (type default))
-  )
-  (wire (pts (xy 124.46 77.47) (xy 124.46 68.58))
-    (stroke (width 0) (type default))
-  )
-  (wire (pts (xy 107.95 77.47) (xy 107.95 80.01))
-    (stroke (width 0) (type default))
-  )
-  (wire (pts (xy 124.46 90.17) (xy 124.46 87.63))
-    (stroke (width 0) (type default))
-  )
-  (wire (pts (xy 124.46 26.035) (xy 96.52 26.035))
-    (stroke (width 0) (type default))
-  )
-  (wire (pts (xy 107.95 77.47) (xy 124.46 77.47))
-    (stroke (width 0) (type default))
-  )
-  (wire (pts (xy 96.52 26.035) (xy 96.52 31.75))
-    (stroke (width 0) (type default))
-  )
-  (wire (pts (xy 62.23 26.035) (xy 74.93 26.035))
     (stroke (width 0) (type default))
   )
@@
     )
   )
+  (symbol (lib_id "Device:D_Zener") (at 124.46 45.72 270) (unit 1)
+    (in_bom yes) (on_board yes) (dnp no) (fields_autoplaced)
+    (property "Reference" "D3" (at 127.635 44.45 90)
+      (effects (font (size 1.27 1.27)) (justify left))
+    )
+    (property "Value" "PZ1AL62B-AU_R1_000A1" (at 127.635 46.99 90)
+      (effects (font (size 1.27 1.27)) (justify left))
+    )
+    (property "Footprint" "Diode_SMD:D_SOD-123F" (at 124.46 45.72 0)
+      (effects (font (size 1.27 1.27)) hide)
+    )
+    (property "Datasheet" "~" (at 124.46 45.72 0)
+      (effects (font (size 1.27 1.27)) hide)
+    )
+    (pin "1")
+    (pin "2")
+    (instances
+      (project "voltage_indicator"
+        (path "/d0262e13-a8ab-42db-962e-1ef7dd9c8d4a"
+          (reference "D3") (unit 1)
+        )
+      )
+    )
+  )
+  (symbol (lib_id "Connector_Generic:Conn_01x02") (at 57.15 28.575 180) (unit 1)
+    (in_bom yes) (on_board yes) (dnp no) (fields_autoplaced)
+    (property "Reference" "Molex2" (at 57.15 19.685 0)
+      (effects (font (size 1.27 1.27)))
+    )
+    (property "Value" "043045-0212" (at 57.15 22.225 0)
+      (effects (font (size 1.27 1.27)))
+    )
+    (property "Footprint" "Connector_Molex:Molex_Micro-Fit_3.0_43045-0212_2x01_P3.00mm_Vertical" (at 57.15 28.575 0)
+      (effects (font (size 1.27 1.27)) hide)
+    )
+    (property "Datasheet" "~" (at 57.15 28.575 0)
+      (effects (font (size 1.27 1.27)) hide)
+    )
+    (pin "1")
+    (pin "2")
+    (instances
+      (project "voltage_indicator"
+        (path "/d0262e13-a8ab-42db-962e-1ef7dd9c8d4a"
+          (reference "Molex2") (unit 1)
+        )
+      )
+    )
+  )
+  (symbol (lib_id "Simulation_SPICE:NJFET") (at 93.98 36.83 0) (unit 1)
+    (in_bom yes) (on_board yes) (dnp no) (fields_autoplaced)
+    (property "Reference" "Q2" (at 99.695 35.56 0)
+      (effects (font (size 1.27 1.27)) (justify left))
+    )
+    (property "Value" "UJ3N120035K3S" (at 99.695 38.1 0)
+      (effects (font (size 1.27 1.27)) (justify left))
+    )
+    (property "Footprint" "Package_TO_SOT_THT:TO-247-3_Horizontal_TabDown" (at 99.06 34.29 0)
+      (effects (font (size 1.27 1.27)) hide)
+    )
+    (property "Datasheet" "~" (at 93.98 36.83 0)
+      (effects (font (size 1.27 1.27)) hide)
+    )
+    (property "Sim.Device" "NJFET" (at 93.98 36.83 0)
+      (effects (font (size 1.27 1.27)) hide)
+    )
+    (property "Sim.Type" "SHICHMANHODGES" (at 93.98 36.83 0)
+      (effects (font (size 1.27 1.27)) hide)
+    )
+    (property "Sim.Pins" "1=D 2=G 3=S" (at 93.98 36.83 0)
+      (effects (font (size 1.27 1.27)) hide)
+    )
+    (pin "1")
+    (pin "2")
+    (pin "3")
+    (instances
+      (project "voltage_indicator"
+        (path "/d0262e13-a8ab-42db-962e-1ef7dd9c8d4a"
+          (reference "Q2") (unit 1)
+        )
+      )
+    )
+  )
   (symbol (lib_id "Device:R") (at 124.46 64.77 0) (unit 1)
-    (in_bom yes) (on_board yes) (dnp no) (fields_autoplaced)
-    (property "Reference" "R3" (at 127 64.135 0)
-      (effects (font (size 1.27 1.27)) (justify left))
-    )
-    (property "Value" "RK73G2BTTD1004C" (at 127 66.675 0)
-      (effects (font (size 1.27 1.27)) (justify left))
-    )
-    (property "Footprint" "Resistor_SMD:RESC3116X65N" (at 122.682 64.77 90)
+    (in_bom yes) (on_board yes) (dnp no)
+    (property "Reference" "R3" (at 126.365 64.135 0)
+      (effects (font (size 1.27 1.27)) (justify left))
+    )
+    (property "Value" "PR02000201004FA100" (at 118.745 69.85 0)
+      (effects (font (size 1.27 1.27)) (justify left))
+    )
+    (property "Footprint" "Resistor_THT:R_Axial_DIN0207_L6.3mm_D2.5mm_P7.62mm_Horizontal" (at 122.682 64.77 90)
       (effects (font (size 1.27 1.27)) hide)
     )
@@
         )
       )
-    )
-  )
-  (symbol (lib_id "Device:D_Zener") (at 124.46 45.72 270) (unit 1)
-    (in_bom yes) (on_board yes) (dnp no) (fields_autoplaced)
-    (property "Reference" "D3" (at 127.635 44.45 90)
-      (effects (font (size 1.27 1.27)) (justify left))
-    )
-    (property "Value" "PZ1AL62B-AU_R1_000A1" (at 127.635 46.99 90)
-      (effects (font (size 1.27 1.27)) (justify left))
-    )
-    (property "Footprint" "Diode_SMD:D_SOD-123F" (at 124.46 45.72 0)
-      (effects (font (size 1.27 1.27)) hide)
-    )
-    (property "Datasheet" "~" (at 124.46 45.72 0)
-      (effects (font (size 1.27 1.27)) hide)
-    )
-    (pin "1")
-    (pin "2")
-    (instances
-      (project "voltage_indicator"
-        (path "/d0262e13-a8ab-42db-962e-1ef7dd9c8d4a"
-          (reference "D3") (unit 1)
-        )
-      )
-    )
-  )
-  (symbol (lib_id "Connector_Generic:Conn_01x02") (at 57.15 28.575 180) (unit 1)
-    (in_bom yes) (on_board yes) (dnp no) (fields_autoplaced)
-    (property "Reference" "Molex2" (at 57.15 19.685 0)
-      (effects (font (size 1.27 1.27)))
-    )
-    (property "Value" "043045-0212" (at 57.15 22.225 0)
-      (effects (font (size 1.27 1.27)))
-    )
-    (property "Footprint" "Connector_Molex:Molex_Micro-Fit_3.0_43045-0212_2x01_P3.00mm_Vertical" (at 57.15 28.575 0)
-      (effects (font (size 1.27 1.27)) hide)
-    )
-    (property "Datasheet" "~" (at 57.15 28.575 0)
-      (effects (font (size 1.27 1.27)) hide)
-    )
-    (pin "1")
-    (pin "2")
-    (instances
-      (project "voltage_indicator"
-        (path "/d0262e13-a8ab-42db-962e-1ef7dd9c8d4a"
-          (reference "Molex2") (unit 1)
-        )
-      )
-    )
-  )
-  (symbol (lib_id "Simulation_SPICE:NJFET") (at 93.98 36.83 0) (unit 1)
-    (in_bom yes) (on_board yes) (dnp no) (fields_autoplaced)
-    (property "Reference" "Q2" (at 99.695 35.56 0)
-      (effects (font (size 1.27 1.27)) (justify left))
-    )
-    (property "Value" "UJ3N120035K3S" (at 99.695 38.1 0)
-      (effects (font (size 1.27 1.27)) (justify left))
-    )
-    (property "Footprint" "Package_TO_SOT_THT:TO-247-3_Horizontal_TabDown" (at 99.06 34.29 0)
-      (effects (font (size 1.27 1.27)) hide)
-    )
-    (property "Datasheet" "~" (at 93.98 36.83 0)
-      (effects (font (size 1.27 1.27)) hide)
-    )
-    (property "Sim.Device" "NJFET" (at 93.98 36.83 0)
-      (effects (font (size 1.27 1.27)) hide)
-    )
-    (property "Sim.Type" "SHICHMANHODGES" (at 93.98 36.83 0)
-      (effects (font (size 1.27 1.27)) hide)
-    )
-    (property "Sim.Pins" "1=D 2=G 3=S" (at 93.98 36.83 0)
-      (effects (font (size 1.27 1.27)) hide)
-    )
-    (pin "1")
-    (pin "2")
-    (pin "3")
-    (instances
-      (project "voltage_indicator"
-        (path "/d0262e13-a8ab-42db-962e-1ef7dd9c8d4a"
-          (reference "Q2") (unit 1)
-        )
-      )
