File: Board_n_schem/TSAL/TSALv2.kicad_sch (KiCad schematic)
At the start: 21 parts, among them J1 043045-0412, Q1 BS250P, Q2 BS170, Q3 UJ3N120035K3S, Q4 BS170, U1 H11L1M

Commit message: removed .DS_store
Connections:
- net HV-: now reaches D1.2 (A), Molex1.1 (Pin_1), Q3.1 (G), Q4.3 (S), R3.2
- net HV+: now reaches D10.1 (K), Molex1.2 (Pin_2), Q3.2 (D)
