File: Schematics/Electrical_system_rev2/accumulator.kicad_sch (KiCad schematic)
At the start: 17 parts, among them K1 GV24 1BAX, K2 PNC113BDA (NC), K3 P115 BDA, K4 GV24 1BAX, Q1 PMOS, SW5 2843011, U2 IMD, U3 BMS, U4 RSB, U5 Battery, U6 Volt_indic, U7 precharge

Commit message: SDC
Connections:
- net at U5. (Therm): now also F2.1; no longer U3. (Therm)
- new net: U3. (Therm), U5. (Therm) (x4)

Commit message: updating of electrical system
Parts:
- removed SW5: 2843011, symbol Switch:SW_SPST
Connections:
- net GLV-: now also K1.2
- net HVD1: now reaches K1.7, K1.8
- net HVD2: now reaches F1.2
- net at U5. (Therm): now also F2.1; no longer U3. (Therm)
- new net: U3. (Therm), U5. (Therm) (x4)

Commit message: swapped male and female connectors
Connections:
- net at U5. (Therm): now also F2.1; no longer U3. (Therm)
- new net: U3. (Therm), U5. (Therm) (x4)

Commit message: updated numberings
Parts:
- renumbered F3 to F1
Connections:
- net at U5. (Therm): now also F2.1; no longer U3. (Therm)
- new net: U3. (Therm), U5. (Therm) (x4)
Changed lines of the file:
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@@
 			(project "Electrical_system_rev2"
 				(path "/e737253b-bf2e-46db-bb95-366ad16822f4/df251301-8247-4edd-baa4-d558109a423b"
-					(reference "U10")
+					(reference "U19")
 					(unit 1)
 				)
@@
 			(project "Electrical_system_rev2"
 				(path "/e737253b-bf2e-46db-bb95-366ad16822f4/df251301-8247-4edd-baa4-d558109a423b"
-					(reference "F1")
+					(reference "F2")
 					(unit 1)
 				)
@@
 			(project "Electrical_system_rev2"
 				(path "/e737253b-bf2e-46db-bb95-366ad16822f4/df251301-8247-4edd-baa4-d558109a423b"
-					(reference "U11")
+					(reference "U20")
 					(unit 1)
 				)
@@
 			(project "Electrical_system_rev2"
 				(path "/e737253b-bf2e-46db-bb95-366ad16822f4/df251301-8247-4edd-baa4-d558109a423b"
-					(reference "F2")
+					(reference "F3")
 					(unit 1)
 				)
@@
 			(project "Electrical_system_rev2"
 				(path "/e737253b-bf2e-46db-bb95-366ad16822f4/df251301-8247-4edd-baa4-d558109a423b"
-					(reference "U9")
+					(reference "U15")
 					(unit 1)
 				)
@@
 			(project "Electrical_system_rev2"
 				(path "/e737253b-bf2e-46db-bb95-366ad16822f4/df251301-8247-4edd-baa4-d558109a423b"
-					(reference "U12")
+					(reference "U16")
 					(unit 1)
 				)
@@
 		(dnp no)
 		(fields_autoplaced yes)
-		(property "Reference" "F3"
+		(property "Reference" "F1"
 			(at 313.69 76.835 90)
 			(effects
@@
 			(project "Electrical_system_rev2"
 				(path "/e737253b-bf2e-46db-bb95-366ad16822f4/df251301-8247-4edd-baa4-d558109a423b"
-					(reference "F3")
+					(reference "F1")
 					(unit 1)
 				)
@@
 			(project "Electrical_system_rev2"
 				(path "/e737253b-bf2e-46db-bb95-366ad16822f4/df251301-8247-4edd-baa4-d558109a423b"
-					(reference "U14")
+					(reference "U18")
 					(unit 1)
 				)
@@
 			(project "Electrical_system_rev2"
 				(path "/e737253b-bf2e-46db-bb95-366ad16822f4/df251301-8247-4edd-baa4-d558109a423b"
-					(reference "U13")
+					(reference "U17")
 					(unit 1)
 				)
@@
 			(project "Electrical_system_rev2"
 				(path "/e737253b-bf2e-46db-bb95-366ad16822f4/df251301-8247-4edd-baa4-d558109a423b"
-					(reference "R1")
+					(reference "R5")
 					(unit 1)
 				)
@@
 			(project "Electrical_system_rev2"
 				(path "/e737253b-bf2e-46db-bb95-366ad16822f4/df251301-8247-4edd-baa4-d558109a423b"
-					(reference "D3")
-					(unit 1)
-				)
+					(reference "D6")
+					(unit 1)
+				)

Commit message: small edits
Connections:
- net at U5. (Therm): now also F2.1; no longer U3. (Therm)
- new net: U3. (Therm), U5. (Therm) (x4)
