File: 2024-25/Schematics/Electrical_system/hv_box.kicad_sch (KiCad schematic)
At the start: 0 parts

Commit message: accum and HV box schm
Parts:
- added J9: 33482-4001, symbol Connector:Conn_01x04_Socket
- added K2: PNC113BDA (NC), Relay_THT:Relay_StandexMeder_DIP_LowProfile, symbol Relay:DIPxx-1Axx-11x
- added R1, R2: PWR220T-35-1502J, symbol Device:R_US
- added TP1, TP2, TP3, TP4: TestPoint, symbol Connector:TestPoint
- added U11: ~, symbol FSAE:Emeter
- added U12: TSAL, symbol Random:TSAL
- added U7: RSB, symbol Random:RSB
Connections:
- new net: R2.2, TP3.1
- new net: K2.7, K2.8, U7. (pre_res-)
- new net: R1.2, TP2.1
- new net: J9.3 (Pin_3), U11.3 (CANL)
- new net: J9.4 (Pin_4), U11.4 (CANH)
- new net GLV-: K2.2
- new net GLVMS: J9.1 (Pin_1), TP4.1, U11.1 (GLV+), U12. (RD+)
- new net GND: J9.2 (Pin_2), TP1.1, U11.2 (GLV-), U12. (RD+)
- new net HV+: R2.1, U11. (VSENSE), U12. (RD+), U7. (pre_res-)
- new net HV-: K2.1, K2.14, R1.1, U11. (VSENSE), U12. (RD+)
- new net SDC_in: K2.6
- new net TSAL_GREEN: U12. (RD+)
- new net TSAL_RED: U12. (RD+)
Other:
- note added: "Download Connector"
- note added: "GLVMP"
- note added: "TSMP"
- title: (none) -> SC FormulaE Electrical System
