File: 2024-25/Schematics/Electrical_system/Electrical_system.kicad_sch (KiCad schematic)
At the start: 28 parts, among them J1 DTM04-12PA-L012, J10 DTM04-12PA-L012, J13 DTM04-12PA-L012, J14 DTP04-4P-LE07, J15 DTM06-12SA, J16 DTM04-12PA-L012, J17 1-66399-0, J18 1-66103-8, J19 DT06-4S, J2 DTM06-12SA, J3 UPCR012ALS1, J4 UPCP012ALS2, J5 UPCR012ALS1, J6 UPCP012ALS2, J7 DTM06-12SA, J8 EM30MSD-A(06), J9 DTM06-12SA, SW3 84-5330.0020, SW4 84-5330.0020

Commit message: one more small fix
Parts:
- J17: value 1-66399-0 -> 211102-1
- J18: value 1-66103-8 -> 206429-1
Changed lines of the file:
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@@
 		)
 		(stroke
-			(width 0.508)
+			(width 0)
 			(type default)
 			(color 204 102 0 1)
@@
 			)
 		)
-		(property "Value" "1-66103-8"
+		(property "Value" "206429-1"
 			(at 156.718 179.705 90)
 			(effects
@@
 			)
 		)
-		(property "Value" "1-66399-0"
+		(property "Value" "211102-1"
 			(at 156.972 188.214 90)
 			(effects

Commit message: fixed some wiring
Connections:
- net checkbox/Current: now also J10.5 (Pin_5); no longer J13.5 (Pin_5)
- net at J7.5 (Pin_5): now also J2.5 (Pin_5)
- net Accumulator/GLV+_fans renamed Accumulator/Current
Other:
- sheet Accumulator ports: added Current; removed GLV+_fans
Changed lines of the file:
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@@
 	)
 	(bus_entry
-		(at 86.36 273.05)
-		(size 2.54 2.54)
-		(stroke
-			(width 0)
-			(type default)
-		)
-	)
-	(bus_entry
 		(at 320.675 181.61)
 		(size 2.54 2.54)
@@
 	)
 	(bus_entry
-		(at 88.9 273.05)
-		(size 2.54 2.54)
-		(stroke
-			(width 0)
-			(type default)
-		)
-	)
-	(bus_entry
 		(at 76.2 273.05)
 		(size 2.54 2.54)
@@
 	)
 	(bus_entry
-		(at 83.82 273.05)
-		(size 2.54 2.54)
-		(stroke
-			(width 0)
-			(type default)
-		)
-	)
-	(bus_entry
 		(at 182.88 170.18)
 		(size 2.54 2.54)
@@
 		)
 	)
-	(bus
-		(pts
-			(xy 86.36 275.59) (xy 88.9 275.59)
-		)
-		(stroke
-			(width 0)
-			(type default)
-		)
-	)
 	(wire
 		(pts
@@
 		)
 	)
-	(bus
-		(pts
-			(xy 88.9 275.59) (xy 91.44 275.59)
-		)
-		(stroke
-			(width 0)
-			(type default)
-		)
-	)
 	(wire
 		(pts
@@
 	(wire
 		(pts
-			(xy 88.9 271.145) (xy 88.9 273.05)
-		)
-		(stroke
-			(width 0)
-			(type default)
-		)
-	)
-	(wire
-		(pts
 			(xy 220.98 120.015) (xy 251.46 120.015)
 		)
@@
 	(bus
 		(pts
-			(xy 83.82 275.59) (xy 86.36 275.59)
+			(xy 83.82 275.59) (xy 96.52 275.59)
 		)
 		(stroke
@@
 		)
 	)
+	(wire
+		(pts
+			(xy 57.785 78.105) (xy 57.785 174.625)
+		)
+		(stroke
+			(width 0)
+			(type default)
+		)
+	)
 	(bus
 		(pts
@@
 	(wire
 		(pts
-			(xy 83.82 271.145) (xy 83.82 273.05)
-		)
-		(stroke
-			(width 0)
-			(type default)
-		)
-	)
-	(wire
-		(pts
 			(xy 276.86 203.835) (xy 238.76 203.835)
 		)
@@
 		)
 	)
+	(wire
+		(pts
+			(xy 57.785 189.865) (xy 57.785 190.5)
+		)
+		(stroke
+			(width 0)
+			(type default)
+		)
+	)
 	(bus
 		(pts
@@
 		)
 	)
-	(bus
-		(pts
-			(xy 91.44 275.59) (xy 96.52 275.59)
-		)
-		(stroke
-			(width 0)
-			(type default)
-		)
-	)
 	(wire
 		(pts
@@
 		)
 	)
-	(wire
-		(pts
-			(xy 86.36 271.145) (xy 86.36 273.05)
-		)
-		(stroke
-			(width 0)
-			(type default)
-		)
-	)
 	(bus
 		(pts
@@
 	(wire
 		(pts
-			(xy 84.455 255.27) (xy 84.455 255.905)
-		)
-		(stroke
-			(width 0)
-			(type default)
-		)
-	)
-	(wire
-		(pts
 			(xy 55.245 63.5) (xy 55.245 64.135)
 		)
@@
 			)
 		)
-		(pin "GLV+_fans" input
+		(pin "Current" input
 			(at 57.785 63.5 270)
 			(effects
@@
 		)
 		(pin "Current" input
-			(at 84.455 255.27 270)
+			(at 57.785 190.5 90)
 			(effects
 				(font
 					(size 1.27 1.27)
 				)
-				(justify left)
+				(justify right)
 			)
 		)

Commit message: updates
Parts:
- added J21: DTM04-12PA-L012, symbol Connector:Conn_01x12_Socket
- added J22: DTM06-12SA, symbol Connector:Conn_01x12_Pin
Connections:
- net Accumulator/Control_Pilot: now also J21.2 (Pin_2); no longer J1.1 (Pin_1)
- net Accumulator/Prox_Detect: now also J21.1 (Pin_1); no longer J1.2 (Pin_2)
- net Accumulator/charge_on: now also J21.4 (Pin_4); no longer J1.4 (Pin_4)
- net Accumulator/charge_safe: now also J21.3 (Pin_3); no longer J1.3 (Pin_3)
- no-connect marks 4 -> 3
Other:
- moved on the sheet: B1, BT1, D2, D5, D6, J1, J10, J13, J14, J15, J16, J17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

Commit message: ESF updates
Connections:
- net Accumulator/PC_error: now reaches J21.5 (Pin_5)
Other:
- sheet Accumulator ports: added PC_error; removed none
- sheet Dash ports: added PC_error; removed none
- note added: "open"
Changed lines of the file:
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@@
 	)
 	(no_connect
-		(at 148.59 137.795)
+		(at 120.015 92.075)
 	)
 	(no_connect
-		(at 146.05 137.795)
+		(at 120.015 86.995)
 	)
 	(no_connect
-		(at 151.13 137.795)
+		(at 120.015 89.535)
 	)
 	(bus_entry
@@
 	)
 	(bus_entry
+		(at 399.415 266.065)
+		(size 2.54 2.54)
+		(stroke
+			(width 0)
+			(type default)
+		)
+	)
+	(bus_entry
 		(at 328.295 106.68)
 		(size 2.54 -2.54)
@@
 		)
 	)
+	(bus_entry
+		(at 169.545 332.74)
+		(size 2.54 2.54)
+		(stroke
+			(width 0)
+			(type default)
+		)
+	)
 	(bus
 		(pts
@@
 	(wire
 		(pts
+			(xy 106.68 332.74) (xy 169.545 332.74)
+		)
+		(stroke
+			(width 0)
+			(type default)
+		)
+	)
+	(wire
+		(pts
 			(xy 158.75 137.795) (xy 158.75 234.315)
 		)
@@
 	(bus
 		(pts
-			(xy 399.415 268.605) (xy 421.64 268.605)
+			(xy 399.415 268.605) (xy 401.955 268.605)
 		)
 		(stroke
@@
 		)
 	)
+	(bus
+		(pts
+			(xy 401.955 268.605) (xy 421.64 268.605)
+		)
+		(stroke
+			(width 0)
+			(type default)
+		)
+	)
 	(wire
 		(pts
@@
 	(wire
 		(pts
+			(xy 399.415 258.445) (xy 399.415 266.065)
+		)
+		(stroke
+			(width 0)
+			(type default)
+		)
+	)
+	(wire
+		(pts
 			(xy 240.665 140.335) (xy 264.795 140.335)
 		)
@@
 	(wire
 		(pts
+			(xy 106.68 97.155) (xy 120.015 97.155)
+		)
+		(stroke
+			(width 0)
+			(type default)
+		)
+	)
+	(wire
+		(pts
 			(xy 186.055 138.43) (xy 186.055 140.97)
 		)
@@
 		)
 	)
+	(bus
+		(pts
+			(xy 172.085 335.28) (xy 174.625 335.28)
+		)
+		(stroke
+			(width 0)
+			(type default)
+		)
+	)
 	(wire
 		(pts
@@
 	(wire
 		(pts
+			(xy 106.68 97.155) (xy 106.68 332.74)
+		)
+		(stroke
+			(width 0)
+			(type default)
+		)
+	)
+	(wire
+		(pts
 			(xy 321.31 220.345) (xy 337.185 220.345)
 		)
@@
 		)
 	)
+	(text "open"
+		(exclude_from_sim no)
+		(at 116.586 94.742 0)
+		(effects
+			(font
+				(size 1.27 1.27)
+			)
+		)
+	)
 	(text "40 A-Hr battery"
 		(exclude_from_sim no)
@@
 			)
 		)
+		(pin "PC_error" output
+			(at 133.985 97.155 180)
+			(effects
+				(font
+					(size 1.27 1.27)
+				)
+				(justify left)
+			)
+		)
 		(instances
 			(project "Electrical_system"
@@
 			(effects
 				(font
+					(size 1.27 1.27)
+				)
+				(justify left)
+			)
+		)
+		(pin "PC_error" input
+			(at 399.415 258.445 270)
+			(effects
+				(font

Commit message: ESF fixes + energy meter updates
Parts:
- added J23: 206429-1, symbol Connector:Conn_01x04_Pin
- added J24: 211102-1, symbol Connector:Conn_01x04_Socket
- J4, J6: value UPCP012ALS2 -> UPCP012ALS1
Connections:
- net HV+_bamocar: no longer J18.1 (Pin_1)
- net Accumulator/temp_sense: now reaches J1.3 (Pin_3)
- net Accumulator/temp_GND: now reaches J1.4 (Pin_4)
- net at J7.3 (Pin_3): now also J2.3 (Pin_3)
- net at J7.4 (Pin_4): now also J2.4 (Pin_4)
- net checkbox/temp_sense: now reaches J10.3 (Pin_3)
- net checkbox/temp_GND: now reaches J10.4 (Pin_4)
- net at J18.2 (Pin_2): now also J23.1 (Pin_1)
- new net: J18.1 (Pin_1), J23.2 (Pin_2)
- new net Accumulator/HV+_bamo: J24.2 (Pin_2)
- new net Accumulator/HV+_tsmp: J24.1 (Pin_1)
Other:
- sheet Accumulator ports: added HV+_bamo, HV+_tsmp, temp_GND, temp_sense; removed none
- sheet checkbox ports: added HV+_tsmp, temp_GND, temp_sense; removed none

Commit message: integration cleanups
Connections:
- net Dash/SDC_to_dash: no longer J15.10 (Pin_10)
- net GLV+_bamo: now also J15.4 (Pin_4); no longer J15.5 (Pin_5)
- net checkbox/BMS_ind: now also J16.2 (Pin_2); no longer J16.3 (Pin_3)
- net checkbox/CANH_500: now also J16.7 (Pin_7); no longer J16.8 (Pin_8)
- net checkbox/CANL_500: now also J16.6 (Pin_6); no longer J16.7 (Pin_7)
- net checkbox/CANS_500: now also J16.5 (Pin_5); no longer J16.6 (Pin_6)
- net checkbox/GLV+_bamo: now also J16.4 (Pin_4); no longer J16.5 (Pin_5)
- net checkbox/HV+_tsmp: now also J17.2 (Pin_2)
- net checkbox/IMD_ind: now also J16.3 (Pin_3); no longer J16.4 (Pin_4)
- net checkbox/SDC_to_TSMS: now also J16.8 (Pin_8); no longer J16.9 (Pin_9)
- net checkbox/SDC_to_dash: now also J13.7 (Pin_7); no longer J16.10 (Pin_10)
- net checkbox/TSAL_R: now also J16.1 (Pin_1); no longer J16.2 (Pin_2)
- net checkbox/temp1: now also J16.12 (Pin_12); no longer J16.11 (Pin_11)
- net checkbox/temp2: now also J16.11 (Pin_11); no longer J16.12 (Pin_12)
- net checkbox/BSPD_ok: now reaches J13.8 (Pin_8)
- net at SW4.2 (B): now also J15.8 (Pin_8); no longer J15.9 (Pin_9)
- net Accumulator/HV+_discharge: now reaches J24.3 (Pin_3)
- net at J15.1 (Pin_1): now also D2.1 (K)
- net at J15.2 (Pin_2): now also D6.2 (A); no longer D2.1 (K)
- net at J15.3 (Pin_3): now also D5.2 (A); no longer D6.2 (A)
- net at J18.3 (Pin_3): now also J23.3 (Pin_3)
- net checkbox/HV+_discharge: now reaches J17.3 (Pin_3)
- net Accumulator/HV+_bamo renamed Accumulator/HV+_TSAL
- net checkbox/HV+_bamo renamed checkbox/HV+_TSAL
- new net Cooling/temp_12V: J15.10 (Pin_10)
- new net checkbox/temp12V: J16.10 (Pin_10)
Other:
- sheet Accumulator ports: added HV+_TSAL, HV+_discharge; removed HV+_bamo
- sheet Cooling ports: added temp_12V; removed none
- sheet Dash ports: added none; removed Current
- sheet checkbox ports: added BSPD_ok, HV+_TSAL, HV+_discharge, temp12V; removed HV+_bamo
- moved on the sheet: J14, J19

Commit message: harness updates
Connections:
- net checkbox/CANH_500: now also J13.6 (Pin_6); no longer J16.7 (Pin_7)
- net checkbox/CANL_500: now also J13.5 (Pin_5); no longer J16.6 (Pin_6)
- net Accumulator/HV+_Emeter: now reaches J24.4 (Pin_4)
- net at J18.4 (Pin_4): now also J23.4 (Pin_4)
- net checkbox/HV+_Emeter: now reaches J17.4 (Pin_4)
- net checkbox/CANS_500: no longer names the net of J16.5 (Pin_5)
Other:
- sheet Accumulator ports: added HV+_Emeter; removed none
- sheet checkbox ports: added HV+_Emeter; removed CANS_500
Changed lines of the file:
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@@
 			(width 0)
 			(type default)
-			(color 204 102 0 1)
+			(color 221 133 0 1)
 		)
 	)
@@
 	(wire
 		(pts
+			(xy 248.285 106.68) (xy 248.285 237.49)
+		)
+		(stroke
+			(width 0)
+			(type default)
+			(color 221 133 0 1)
+		)
+	)
+	(wire
+		(pts
 			(xy 171.45 249.555) (xy 171.45 250.19)
 		)
@@
 			(width 0)
 			(type default)
+			(color 221 133 0 1)
 		)
 	)
@@
 	(wire
 		(pts
+			(xy 216.535 106.68) (xy 248.285 106.68)
+		)
+		(stroke
+			(width 0)
+			(type default)
+			(color 221 133 0 1)
+		)
+	)
+	(wire
+		(pts
 			(xy 191.135 142.875) (xy 191.135 234.315)
 		)
@@
 			(width 0)
 			(type default)
+			(color 221 133 0 1)
 		)
 	)
@@
 		)
 	)
+	(wire
+		(pts
+			(xy 185.42 314.96) (xy 185.42 315.595)
+		)
+		(stroke
+			(width 0)
+			(type default)
+		)
+	)
 	(bus
 		(pts
@@
 		)
 	)
+	(wire
+		(pts
+			(xy 203.835 106.68) (xy 204.47 106.68)
+		)
+		(stroke
+			(width 0)
+			(type default)
+		)
+	)
 	(bus
 		(pts
@@
 	(wire
 		(pts
+			(xy 182.88 314.96) (xy 182.88 315.595)
+		)
+		(stroke
+			(width 0)
+			(type default)
+		)
+	)
+	(wire
+		(pts
 			(xy 327.025 229.235) (xy 327.025 288.29)
 		)
@@
 	(wire
 		(pts
+			(xy 248.285 249.555) (xy 248.285 250.19)
+		)
+		(stroke
+			(width 0)
+			(type default)
+			(color 221 133 0 1)
+		)
+	)
+	(wire
+		(pts
 			(xy 168.91 229.87) (xy 168.91 234.315)
 		)
@@
 			(width 0)
 			(type default)
-			(color 204 102 0 1)
+			(color 221 133 0 1)
 		)
 	)
@@
 			)
 		)
+		(pin "HV+_Emeter" output
+			(at 203.835 106.68 0)
+			(effects
+				(font
+					(size 1.27 1.27)
+				)
+				(justify right)
+			)
+		)
 		(instances
 			(project "Electrical_system"
@@
 			)
 		)
-		(pin "CANL_500" bidirectional
-			(at 281.94 250.19 90)
-			(effects
-				(font
-					(size 1.27 1.27)
-				)
-				(justify right)
-			)
-		)
-		(pin "CANH_500" bidirectional
-			(at 284.48 250.19 90)
-			(effects
-				(font
-					(size 1.27 1.27)
-				)
-				(justify right)
-			)
-		)
-		(pin "CANS_500" bidirectional
-			(at 279.4 250.19 90)
-			(effects
-				(font
-					(size 1.27 1.27)
-				)
-				(justify right)
-			)
-		)
 		(pin "SDC_to_TSMS" input
 			(at 287.02 250.19 90)
@@
 			(effects
 				(font
+					(size 1.27 1.27)
+				)
+				(justify right)
+			)
+		)
+		(pin "CANL_500" bidirectional
+			(at 182.88 314.96 270)
+			(effects
+				(font
+					(size 1.27 1.27)
+				)
+				(justify left)
+			)
+		)
+		(pin "CANH_500" bidirectional
+			(at 185.42 314.96 270)
+			(effects
+				(font
+					(size 1.27 1.27)
+				)
+				(justify left)
+			)
+		)
+		(pin "HV+_Emeter" input
+			(at 248.285 250.19 90)
+			(effects
+				(font

Commit message: harness changes
Connections:
- net checkbox/GLV+_lights: now reaches J16.5 (Pin_5)
- net checkbox/BMS_ind renamed checkbox/ind_Green
- net checkbox/IMD_ind renamed checkbox/ind_Red
Other:
- sheet checkbox ports: added GLV+_lights, ind_Green, ind_Red; removed BMS_ind, IMD_ind
Changed lines of the file:
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@@
 		(color 132 0 0 1)
 	)
-	(junction
-		(at 278.765 184.15)
-		(diameter 0)
-		(color 0 0 0 0)
-	)
 	(no_connect
 		(at 120.015 92.075)
@@
 	)
 	(bus_entry
-		(at 278.765 229.87)
-		(size 2.54 2.54)
-		(stroke
-			(width 0)
-			(type default)
-		)
-	)
-	(bus_entry
 		(at 189.865 332.74)
 		(size 2.54 2.54)
@@
 	)
 	(bus_entry
-		(at 281.305 229.87)
-		(size 2.54 2.54)
-		(stroke
-			(width 0)
-			(type default)
-		)
-	)
-	(bus_entry
 		(at 325.755 106.68)
 		(size 2.54 -2.54)
@@
 		)
 	)
-	(bus
-		(pts
-			(xy 278.765 184.15) (xy 278.765 229.87)
-		)
-		(stroke
-			(width 0)
-			(type default)
-			(color 132 0 132 1)
-		)
-	)
 	(wire
 		(pts
@@
 	(bus
 		(pts
-			(xy 278.765 184.15) (xy 351.155 184.15)
+			(xy 254 184.15) (xy 351.155 184.15)
 		)
 		(stroke
@@
 	(wire
 		(pts
-			(xy 281.305 232.41) (xy 281.305 234.315)
-		)
-		(stroke
-			(width 0)
-			(type default)
-		)
-	)
-	(wire
-		(pts
 			(xy 153.67 249.555) (xy 153.67 250.19)
 		)
@@
 		)
 	)
-	(bus
-		(pts
-			(xy 278.765 229.87) (xy 281.305 229.87)
-		)
-		(stroke
-			(width 0)
-			(type default)
-			(color 132 0 132 1)
-		)
-	)
 	(wire
 		(pts
@@
 	(wire
 		(pts
-			(xy 283.845 232.41) (xy 283.845 234.315)
-		)
-		(stroke
-			(width 0)
-			(type default)
-		)
-	)
-	(wire
-		(pts
 			(xy 303.53 201.295) (xy 311.15 201.295)
 		)
@@
 	(bus
 		(pts
-			(xy 254 184.15) (xy 278.765 184.15)
-		)
-		(stroke
-			(width 0)
-			(type default)
-			(color 132 0 132 1)
-		)
-	)
-	(bus
-		(pts
 			(xy 202.565 335.28) (xy 384.81 335.28)
 		)
@@
 	(wire
 		(pts
-			(xy 278.765 229.87) (xy 278.765 234.315)
-		)
-		(stroke
-			(width 0)
-			(type default)
-		)
-	)
-	(wire
-		(pts
 			(xy 286.385 220.345) (xy 286.385 234.315)
 		)
@@
 			)
 		)
-		(pin "IMD_ind" input
+		(pin "ind_Red" input
 			(at 274.32 250.19 90)
 			(effects
@@
 			)
 		)
-		(pin "BMS_ind" input
+		(pin "ind_Green" input
 			(at 271.78 250.19 90)
 			(effects
@@
 			(effects
 				(font
+					(size 1.27 1.27)
+				)
+				(justify right)
+			)
+		)
+		(pin "GLV+_lights" input
+			(at 279.4 250.19 90)
+			(effects
+				(font
