File: 2024-25/Boards/Fab_assembly/Fab_assembly.kicad_pcb (KiCad board)
At the start: 2 copper layers, 0 parts

Commit message: checkbox schm
Parts:
- added C3: 10uF, Capacitor_SMD:C_1206_3216Metric_Pad1.33x1.80mm_HandSolder, F.Cu at (79.9, 63.9)
- added D1: BZT52-B12_R1_00001, Diode_SMD:D_SOD-123, F.Cu at (127.6, 72.4)
- added D2: PZ1AL62B-AU_R1_000A1, Diode_SMD:D_SOD-123F, F.Cu at (147.8, 72.8)
- added D20: PD3S0230, Diode_SMD:D_SOD-110, F.Cu at (88.7, 74.8)
- added D21: 1N4148WX-TP, Diode_SMD:D_SOD-323, F.Cu at (85.7, 70.0)
- added D22: 1N4148WX-TP, Diode_SMD:D_SOD-323, F.Cu at (88.7, 77.3)
- added F1: 750mA, BK_PCS:FUSE_BK_PCS, F.Cu at (151.8, 67.0)
- added H1: MountingHole, MountingHole:MountingHole_4.3mm_M4, F.Cu at (117.8, 55.8)
- added H2: MountingHole, MountingHole:MountingHole_4.3mm_M4, F.Cu at (153.8, 56.0)
- added H3: MountingHole, MountingHole:MountingHole_4.3mm_M4, F.Cu at (117.8, 97.0)
- added H4: MountingHole, MountingHole:MountingHole_4.3mm_M4, F.Cu at (153.8, 97.0)
- added H5: MountingHole, MountingHole:MountingHole_4.3mm_M4, F.Cu at (70.5, 57.1)
- added H6: MountingHole, MountingHole:MountingHole_4.3mm_M4, F.Cu at (106.0, 57.1)
- added H7: MountingHole, MountingHole:MountingHole_4.3mm_M4, F.Cu at (106.0, 77.8)
- added H8: MountingHole, MountingHole:MountingHole_4.3mm_M4, F.Cu at (70.5, 77.8)
- added J3: Conn_01x08, Connector_Molex:Molex_Micro-Fit_3.0_43045-0812_2x04_P3.00mm_Vertical, F.Cu at (80.8, 55.4)
- added Molex1: 043045-0212, Connector_Molex:Molex_Micro-Fit_3.0_43045-0212_2x01_P3.00mm_Vertical, F.Cu at (127.3, 55.9)
- added Molex2: 043045-0212, Connector_Molex:Molex_Micro-Fit_3.0_43045-0212_2x01_P3.00mm_Vertical, F.Cu at (143.7, 55.5)
- added Q1: UJ3N120035K3S, Package_TO_SOT_THT:TO-247-3_Horizontal_TabDown, F.Cu at (125.8, 78.8)
- added Q10: VP3203N8-G, VP3203N8-G:TO-243AA_MCH, F.Cu at (98.1, 55.2)
- added Q11: VN3205N3-G, VN3205N8-G:TO-243AA_MCH, F.Cu at (95.1, 75.3)
- added Q12: VP3203N8-G, VP3203N8-G:TO-243AA_MCH, F.Cu at (87.0, 65.6)
- added Q16: VP3203N8-G, VP3203N8-G:TO-243AA_MCH, F.Cu at (95.3, 69.5)
- added Q2: VN2460, Package_TO_SOT_THT:TO-92, F.Cu at (137.0, 56.9)
- added R1: 1100, Resistor_THT:R_Axial_DIN0207_L6.3mm_D2.5mm_P7.62mm_Horizontal, F.Cu at (121.5, 73.9)
- added R10: 10k, Resistor_SMD:R_0805_2012Metric_Pad1.20x1.40mm_HandSolder, F.Cu at (96.5, 60.3)
- added R12: 1.8M, Resistor_SMD:R_0805_2012Metric_Pad1.20x1.40mm_HandSolder, F.Cu at (85.9, 72.5)
- added R13: 10k, Resistor_SMD:R_0805_2012Metric_Pad1.20x1.40mm_HandSolder, F.Cu at (79.8, 69.5)
- added R17: 10k, Resistor_SMD:R_0805_2012Metric_Pad1.20x1.40mm_HandSolder, F.Cu at (91.2, 67.5)
- added R17: 10k, Resistor_SMD:R_0805_2012Metric_Pad1.20x1.40mm_HandSolder, F.Cu at (79.9, 67.1)
- added R2: PR02000201004FA100, Resistor_THT:R_Axial_DIN0207_L6.3mm_D2.5mm_P7.62mm_Horizontal, F.Cu at (145.9, 68.1)
- added R3: RK73G2BTTD1004C, Resistor_SMD:RESC3116X65N, F.Cu at (127.3, 67.2)
- added R6: 10k, Resistor_SMD:R_0805_2012Metric_Pad1.20x1.40mm_HandSolder, F.Cu at (85.2, 76.0)
- added U3: LM358DR2G, Package_SO:SOIC-8_3.9x4.9mm_P1.27mm, F.Cu at (80.5, 75.0)
Routing:
- net (no net): track 0.00 -> 102.5 mm, vias 0 -> 5
- net Net-(D3-K): track 0.00 -> 39.5 mm
- net /opamp_out: track 0.00 -> 37.5 mm, vias 0 -> 2
- net Vcc: track 0.00 -> 36.6 mm
- net AIR+_en: track 0.00 -> 30.4 mm
- net Net-(D2-K): track 0.00 -> 26.2 mm
- net SDCin: track 0.00 -> 24.7 mm, vias 0 -> 2
- net /RC_timer: track 0.00 -> 20.8 mm
- net CHG: track 0.00 -> 20.5 mm
- net charge_on: track 0.00 -> 18.1 mm
- net /opamp_out_inv: track 0.00 -> 12.9 mm
- net PreAIR_en: track 0.00 -> 12.3 mm, vias 0 -> 2
- net /LED+: track 0.00 -> 9.75 mm
- net Net-(D1-K): track 0.00 -> 8.03 mm
- net /LED-: track 0.00 -> 7.57 mm
- added copper zone on B.Cu, net (none)
Other:
- board outline added: 94.5 x 53.3 mm
- board text added: "Pre/Discharge"
- board text added: "SCFormulaE-"
- board text added: "Voltage Indicator Light"
