File: 2024-25/Boards/Fab_assembly/Fab_assembly.kicad_sch (KiCad schematic)
At the start: 81 parts, among them J1 043045-0412, J2 043045-1212, J3 Conn_01x06, J4 043045-1212, K1 1462043-4, K2 1462043-4, K3 1462043-4, K4 1462043-4, K5 1462043-4, K6 1462043-4, K7 1462043-4, K8 1462043-4, Q1 UJ3N120035K3S, Q10 VN3205N3-G, Q11 VP3203N3-G, Q12 VP3203N3-G, Q13 PJA3412_R1_00001, Q14 PJA3412_R1_00001, Q15 PJA3412_R1_00001, Q2 VN2460, Q3 UJ3N120035K3S, Q4 BS170, Q5 BS170, Q6 BS250P, Q7 PJA3412_R1_00001, Q8 PJA3412_R1_00001, Q9 PJA3412_R1_00001, U1 H11L1M, U2 HEF4049B, U3 LM358DR2G, U4 HEF4049B

Commit message: checkbox schm
Parts:
- removed C1: 10uF, Capacitor_THT:CP_Radial_D4.0mm_P2.00mm, symbol Device:C_Polarized
- removed D23, D24, D25, D26, D27, D28, D29: 1N4148, Diode_THT:D_DO-35_SOD27_P7.62mm_Horizontal, symbol Diode:1N4148
- removed J2: 043045-1212, Connector_Molex:Molex_Micro-Fit_3.0_43045-1212_2x06_P3.00mm_Vertical, symbol Connector_Generic:Conn_01x12
- removed J3: Conn_01x06, Connector_Molex:Molex_Micro-Fit_3.0_43045-0612_2x03_P3.00mm_Vertical, symbol Connector_Generic:Conn_01x06
- removed K5, K6, K7, K8: 1462043-4, Relay_SMD:Relay_DPDT_AXICOM_IMSeries_JLeg, symbol Relay:RT44xxxx
- removed Q10: VN3205N3-G, Package_TO_SOT_THT:TO-92_Inline, symbol Transistor_FET:BS170
- removed Q11, Q12: VP3203N3-G, Package_TO_SOT_THT:TO-92_Inline, symbol Transistor_FET:BS250
- removed Q13, Q14, Q15: PJA3412_R1_00001, Package_TO_SOT_SMD:SOT-23, symbol Transistor_FET:BUK7M8R0-40EX
- removed R10, R15, R16: 10k, Resistor_THT:R_Axial_DIN0207_L6.3mm_D2.5mm_P7.62mm_Horizontal, symbol Device:R_US
- removed U4: HEF4049B, Package_SO:SO-16_3.9x9.9mm_P1.27mm, symbol Random:HEF4049B
- added C1, C4, C6: 1uF, Capacitor_SMD:C_0805_2012Metric_Pad1.18x1.45mm_HandSolder, symbol Device:C
- added C2, C5: .1uF, Capacitor_SMD:C_0603_1608Metric_Pad1.08x0.95mm_HandSolder, symbol Device:C
- added C3: 10uF, Capacitor_SMD:C_1206_3216Metric_Pad1.33x1.80mm_HandSolder, symbol Device:C_Polarized
- added C7: .1uF, Capacitor_SMD:C_0201_0603Metric_Pad0.64x0.40mm_HandSolder, symbol Device:C
- added H1, H10, H11, H12, H13, H14, H15, H16, H2, H3, H4, H5, H6, H7, H8, H9: MountingHole, MountingHole:MountingHole_4.3mm_M4, symbol Mechanical:MountingHole
- added J3: Conn_01x08, Connector_Molex:Molex_Micro-Fit_3.0_43045-0812_2x04_P3.00mm_Vertical, symbol Connector_Generic:Conn_01x08
- added Q10, Q12, Q16: VP3203N8-G, VP3203N8-G:TO-243AA_MCH, symbol Simulation_SPICE:PMOS
- added Q11: VN3205N3-G, VN3205N8-G:TO-243AA_MCH, symbol Transistor_FET:BS170
- added R10: 10k, Resistor_SMD:R_0805_2012Metric_Pad1.20x1.40mm_HandSolder, symbol Device:R_Small_US
- added R17: 10k, Resistor_SMD:R_0805_2012Metric_Pad1.20x1.40mm_HandSolder, symbol Device:R_US
- D21, D22: value 1N4148WTQ-7 -> 1N4148WX-TP; footprint Diode_SMD:D_SOD-523 -> Diode_SMD:D_SOD-323
- R11: value 1.8M -> 10k; footprint Resistor_THT:R_Axial_DIN0207_L6.3mm_D2.5mm_P7.62mm_Horizontal -> Resistor_SMD:R_0805_2012Metric_Pad1.20x1.40mm_HandSolder
- R12: value 10k -> 1.8M; footprint Resistor_THT:R_Axial_DIN0207_L6.3mm_D2.5mm_P7.62mm_Horizontal -> Resistor_SMD:R_0805_2012Metric_Pad1.20x1.40mm_HandSolder
- R13, R14: footprint Resistor_THT:R_Axial_DIN0207_L6.3mm_D2.5mm_P7.62mm_Horizontal -> Resistor_SMD:R_0805_2012Metric_Pad1.20x1.40mm_HandSolder
Connections:
- net BMS Fault: now also J4.8 (Pin_8); no longer J4.6 (Pin_6)
- net BMS_charge: no longer J4.12 (Pin_12)
- net BMS_indicator: now also J4.3 (Pin_3); no longer J4.10 (Pin_10)
- net BMS_power: no longer J4.11 (Pin_11)
- net BSPD Fault: now also J4.6 (Pin_6); no longer J4.8 (Pin_8)
- net GND: now also C6.2, C7.2; no longer D19.2 (A), D22.2 (A), J4.2 (Pin_2), K4.8, Q7.2 (S), Q7.3 (S), Q8.2 (S), Q8.3 (S), Q9.2 (S), Q9.3 (S), R13.1, R8.2, U2.8 (Vss), U3.4 (Vee/GND)
- net IMD Fault: now also J4.1 (Pin_1); no longer J4.7 (Pin_7)
- net SDCin: now also C1.1, C2.1, J3.6 (Pin_6), Q12.3 (S), Q16.3 (S)
- net SW: no longer J4.5 (Pin_5)
- net Vcc: now also R13.1, R17.2; no longer R12.1, R14.2, U3.8 (VCC)
- net opamp_out: now also Q11.1 (G), Q12.2 (G)
- net opamp_out_inv: now also Q11.2 (D), Q16.2 (G), R17.1; no longer R14.1
- net RC_timer: now reaches D21.2 (A), D22.1 (K), U3.5 (IN_B+)
- net RC_timer: now also R12.1, C3.1; no longer R11.1
- net at R13.2, U3.6 (IN_B-): now also R14.2; no longer R12.2
- net at D20.1 (K), D21.1 (K), R11.2: now also R12.2
- net +12V renamed Vcc_relay1
- net Vcc_relay1: now also C4.1, C5.1; no longer J4.1 (Pin_1), K4.6, U2.1 (Vdd)
- net GLV+ renamed GLV+_TSAL
- net GLV- renamed GLV-_TSAL
- net HV+ renamed HV+_TSAL
- net HV+_TSAL: no longer F1.1, Molex1.2 (Pin_2)
- net HV- renamed HV-_TSAL
- net HV-_TSAL: no longer D1.2 (A), Molex1.1 (Pin_1), Q1.1 (G), Q2.1 (S), R3.2
- net SDC 1 renamed SDC1
- net SDC1: now also J4.10 (Pin_10); no longer J4.3 (Pin_3)
- net SDC 2 renamed SDC2
- new net AIR+_en: J3.3 (Pin_3), Q10.3 (S), Q16.1 (D), R10.1
- new net CHG: J3.1 (Pin_1), Q10.1 (D)
- new net GND_PC: C1.2, C2.2, C3.2, D22.2 (A), J3.5 (Pin_5), Q11.3 (S), R11.1, R14.1, U3.4 (Vee/GND)
- new net GND_relay: C4.2, C5.2, D19.2 (A), J4.2 (Pin_2), K4.8, Q7.2 (S), Q7.3 (S), Q8.2 (S), Q8.3 (S), Q9.2 (S), Q9.3 (S), R8.2, U2.8 (Vss)
- new net HV+_VIL: F1.1, Molex1.2 (Pin_2)
- new net HV-_VIL: D1.2 (A), Molex1.1 (Pin_1), Q1.1 (G), Q2.1 (S), R3.2
- new net PreAIR_en: J3.4 (Pin_4), Q12.1 (D)
- new net Reset: J4.5 (Pin_5)
- new net Vcc_PC: J3.7 (Pin_7), U3.8 (VCC)
- new net Vcc_relay: C6.1, C7.1, J4.7 (Pin_7), K4.6, U2.1 (Vdd)
- new net charge_on: J3.2 (Pin_2), Q10.2 (G), R10.2
- no-connect marks 20 -> 11
Other:
- note added: "Input filter"
- note added: "Input filters"
- note added: "Set BMS to charging mode not part of Precharge but we just stuck it on this board XD"
