File: 2024-25/Schematics/Charging/_autosave-Charging_updated.kicad_sch (KiCad schematic)
At the start: 32 parts, among them J1 DTM04-12PA-L012, J2 DTM06-12SA, J3 DTM06-12SA, J4 DTM04-12PA-L012, J5 UPCP012ALS2, J6 UPCR012ALS1, J7 UPCR012ALS1, J8 UPCP012ALS2, K1 GV24 1BAX, K2 Relay_DPST-NO, K3 P115 BDA, K4 GV24 1BAX, SW1 84-5330.0020, U2 Relay board, U3 BMS, U4 6.6kW Elcon Charger, U5 RSB, U6 Throttle, U7 Volt_indic, U8 precharge

Commit message: updates
Connections:
- net CANS_BMS is gone; now on net CANGND_BMS: J2.6 (Pin_6), J3.6 (Pin_6)
- net BMS_fault: now also J1.3 (Pin_3)
- net CANH_BMS: now also J1.5 (Pin_5)
- net CANL_BMS: now also J1.4 (Pin_4)
- net CSS: no longer J1.1 (Pin_1)
- net GLV+: now also J1.9 (Pin_9)
- net GND: now also U2. (SW)
- net GNDPWR: now also J1.10 (Pin_10)
- net IMD_fault: now also J1.2 (Pin_2)
- net at K2.14: now also U4. (Output-)
- net at K2.24: now also U4. (Output-)
- net at U6. (Therm): no longer U3. (Therm)
- net CANGND_BMS: now reaches J1.6 (Pin_6)
- net at J6.3 (Pin_3), R1.1: now also U4. (Output-)
- net at J6.4 (Pin_4), R2.1: now also U4. (Output-)
- net at U5. (pre_res-): now also K3.7, K3.8
- net 12V+: no longer names the net of J4.8 (Pin_8)
- net 12V+: no longer U4.10 (12V5)
- new net: U3. (Therm), U6. (Therm) (x4)
- now unconnected: U6. (Therm), U6. (Therm), U6. (Therm)
Other:
- note added: "(12V 5A o/p no longer used)"
- note added: "external AC connector (i/p)"
- note added: "when CSS (active high) turns on, relay turns off Kill switch to the charger"
- moved on the sheet: F1, F2, J1, U3, U4
