File: 2025-26/Schematics/accumulator_25-26_testSetup/accumulator_charging_testSetup/Accumulator Test Setup-backups/Accumulator Test Setup-2025-09-08_211909/accumulator_charging_testSetup.kicad_sch (KiCad schematic)
At the start: 10 parts, among them J20 ??? can't find PN, K1 RC-400012-DS (Mock), K2 R51−1D70−12F (Mock), K3 GV24 1BAX, SW1 HV Disconnect (Mock), SW2 E-Stop, U16 Battery Segment, U18 BMS, U4 6.6kW Elcon Charger

Commit message: .
Connections:
- net CANH: no longer U4.1 (CANH)
- net CANL: no longer U4.7 (CANL)
- net CANS: now also U18.17 (C1S)
- net at U16. (14-pin_Connector): no longer U18. (GND_Lug)
- new net: U16. (14-pin_Connector), U18. (GND_Lug) (x2)
- now unconnected: U16. (14-pin_Connector)
Other:
- moved on the sheet: K3, U16, U4
Changed lines of the file:
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@@
+		)
+	)
+	(bus_entry
+		(at 47.625 123.19)
+		(size -2.54 2.54)
+		(stroke
+			(width 0)
+			(type default)
+		)
+	)
+	(bus_entry
+		(at 47.625 118.11)
+		(size -2.54 2.54)
+		(stroke
+			(width 0)
+			(type default)
+		)
+	)
+	(bus_entry
+		(at 47.625 120.65)
+		(size -2.54 2.54)
+		(stroke
+			(width 0)
+			(type default)
 		)
 	)
@@
 		)
 	)
-	(wire
-		(pts
-			(xy 46.99 120.65) (xy 53.34 120.65)
+	(bus
+		(pts
+			(xy 45.085 120.65) (xy 45.085 123.19)
+		)
+		(stroke
+			(width 0)
+			(type default)
+		)
+	)
+	(wire
+		(pts
+			(xy 47.625 123.19) (xy 53.34 123.19)
+		)
+		(stroke
+			(width 0)
+			(type default)
+		)
+	)
+	(wire
+		(pts
+			(xy 47.625 118.11) (xy 53.34 118.11)
 		)
 		(stroke
@@
 	(wire
 		(pts
-			(xy 46.99 120.65) (xy 46.99 181.61)
-		)
-		(stroke
-			(width 0)
-			(type default)
-		)
-	)
-	(wire
-		(pts
-			(xy 165.1 129.54) (xy 163.83 129.54)
-		)
-		(stroke
-			(width 0)
-			(type default)
-		)
-	)
-	(wire
-		(pts
 			(xy 82.55 110.49) (xy 82.55 93.98)
 		)
@@
 	(wire
 		(pts
-			(xy 163.83 180.34) (xy 45.72 180.34)
-		)
-		(stroke
-			(width 0)
-			(type default)
-		)
-	)
-	(wire
-		(pts
 			(xy 116.205 133.35) (xy 135.255 133.35)
 		)
@@
 	(wire
 		(pts
-			(xy 91.44 87.63) (xy 109.22 87.63)
+			(xy 91.44 87.63) (xy 110.49 87.63)
 		)
 		(stroke
@@
 	(wire
 		(pts
-			(xy 45.72 180.34) (xy 45.72 118.11)
-		)
-		(stroke
-			(width 0)
-			(type default)
-		)
-	)
-	(wire
-		(pts
-			(xy 46.99 181.61) (xy 165.1 181.61)
-		)
-		(stroke
-			(width 0)
-			(type default)
-		)
-	)
-	(wire
-		(pts
-			(xy 82.55 93.98) (xy 109.22 93.98)
+			(xy 82.55 93.98) (xy 110.49 93.98)
 		)
 		(stroke
@@
 		)
 	)
-	(wire
-		(pts
-			(xy 45.72 118.11) (xy 53.34 118.11)
-		)
-		(stroke
-			(width 0)
-			(type default)
-		)
-	)
-	(wire
-		(pts
-			(xy 163.83 129.54) (xy 163.83 180.34)
-		)
-		(stroke
-			(width 0)
-			(type default)
-		)
-	)
-	(wire
-		(pts
-			(xy 53.34 138.43) (xy 52.705 138.43)
-		)
-		(stroke
-			(width 0)
-			(type default)
-		)
-	)
-	(wire
-		(pts
-			(xy 165.1 181.61) (xy 165.1 132.08)
+	(bus
+		(pts
+			(xy 45.085 123.19) (xy 45.085 125.73)
+		)
+		(stroke
+			(width 0)
+			(type default)
+		)
+	)
+	(bus
+		(pts
+			(xy 45.085 125.73) (xy 45.085 176.53)
+		)
+		(stroke
+			(width 0)
+			(type default)
+		)
+	)
+	(wire
+		(pts
+			(xy 53.34 138.43) (xy 55.245 138.43)
+		)
+		(stroke
+			(width 0)
+			(type default)
+		)
+	)
+	(wire
+		(pts
+			(xy 47.625 120.65) (xy 53.34 120.65)
 		)
 		(stroke
@@
 	(global_label "CONTROL_PILOT"
 		(shape input)
-		(at 52.705 138.43 180)
-		(fields_autoplaced yes)
-		(effects
-			(font
-				(size 1.27 1.27)
-			)
-			(justify right)
-		)
-		(property "Intersheetrefs" "${INTERSHEET_REFS}"
-			(at 35.024 138.43 0)
+		(at 55.245 138.43 180)
+		(fields_autoplaced yes)
+		(effects
+			(font
+				(size 1.27 1.27)
+			)
+			(justify right)
+		)
+		(property "Intersheetrefs" "${INTERSHEET_REFS}"
+			(at 37.564 138.43 0)
 			(effects
 				(font
@@
 	(symbol
 		(lib_id "Accumulator Charging:DIPxx-1Axx-11x")
-		(at 134.62 49.53 270)
+		(at 152.4 41.91 0)
 		(unit 1)
 		(exclude_from_sim no)
@@
 		(dnp no)
 		(property "Reference" "K3"
-			(at 132.842 34.544 90)
+			(at 160.655 40.64 0)
 			(effects
 				(font
@@
 		)
 		(property "Value" "GV24 1BAX"
-			(at 129.286 37.084 90)
+			(at 147.32 48.895 0)
 			(effects
 				(font
@@
 		)
 		(property "Footprint" "Relay_THT:Relay_StandexMeder_DIP_LowProfile"
-			(at 133.35 58.42 0)
+			(at 161.29 43.18 0)
 			(effects
 				(font
@@
 		)
 		(property "Datasheet" "https://www.sensata.com/sites/default/files/a/sensata-gigavac-gv24-sereies-800v-contactors-datasheet.pdf"
-			(at 134.62 49.53 0)
+			(at 152.4 41.91 0)
 			(effects
 				(font
@@
 		)
 		(property "Description" ""
-			(at 134.62 49.53 0)
+			(at 152.4 41.91 0)
 			(effects
 				(font
@@
 		(lib_name "Elcon_1")
 		(lib_id "Accumulator Charging:Elcon")
-		(at 183.515 77.47 180)
+		(at 184.15 77.47 180)
 		(unit 1)
 		(exclude_from_sim no)
@@
 		(dnp no)
 		(property "Reference" "U4"
-			(at 183.388 138.684 0)
+			(at 184.023 138.684 0)
 			(effects
 				(font
@@
 		)
 		(property "Value" "6.6kW Elcon Charger"
-			(at 182.626 99.06 0)
+			(at 183.261 99.06 0)
 			(effects
 				(font
@@
 		)
 		(property "Footprint" ""
-			(at 183.515 77.47 0)
+			(at 184.15 77.47 0)
 			(effects
 				(font
@@
 		)
 		(property "Datasheet" "https://drive.google.com/file/d/1VmoDZTyT_GKdlcjNlQDRAciwgWTCW6jb/view"
-			(at 183.515 77.47 0)
+			(at 184.15 77.47 0)
 			(effects
 				(font
@@
 		)
 		(property "Description" ""
-			(at 183.515 77.47 0)
+			(at 184.15 77.47 0)
 			(effects
 				(font
@@
 		(lib_name "Battery_1")
 		(lib_id "Accumulator Charging:Battery")
-		(at 125.73 77.47 180)
+		(at 127 77.47 180)
 		(unit 1)
 		(exclude_from_sim no)
@@
 		(dnp no)
 		(property "Reference" "U16"
-			(at 127.508 79.502 0)
+			(at 128.778 79.502 0)
 			(effects
 				(font
@@
 		)
 		(property "Value" "Battery Segment"
-			(at 125.73 77.47 0)
+			(at 127 77.47 0)
 			(effects
 				(font
@@
 		)
 		(property "Footprint" ""
-			(at 125.73 77.47 0)
+			(at 127 77.47 0)
 			(effects
 				(font
@@
 		)
 		(property "Datasheet" ""
-			(at 125.73 77.47 0)
+			(at 127 77.47 0)
 			(effects
 				(font
@@
 		)
 		(property "Description" ""
-			(at 125.73 77.47 0)
-			(effects
-				(font
+			(at 127 77.47 0)
+			(effects
+				(font
