File: 2025-26/Boards/RelayBoard/relayBoard.kicad_sch (KiCad schematic)
At the start: 70 parts, among them J1 043045-1212, J2 Conn_01x04_Pin, K4 HF42F/012-2HST, K5 HF42F/012-2HST, K6 HF42F/012-2HST, K7 HF42F/012-2HST, Q1 AO3400A, Q10 AO3400A, Q11 AO3400A, Q2 AO3400A, Q3 AO3401A, Q4 AO3400A, Q5 AO3400A, Q6 AO3401A, Q7 AO3400A, Q9 AO3400A, U4 UA78M33QDCYRQ1, U5 STM32C011F4Px

Commit message: relay board revision
Parts:
- removed D12, D7: PESD5V0S1UL, Diode_SMD:D_SOD-882, symbol Diode:PESD5V0S1UL
- removed D19: PSM712-LF-T7, Package_TO_SOT_SMD:SOT-23, symbol easyeda2kicad:PSM712-LF-T7
- removed R3: 330, Resistor_SMD:R_0603_1608Metric, symbol Device:R_US
- added R25: 47, Resistor_SMD:R_0603_1608Metric, symbol Device:R_US
- added R26, R27: 100k, Resistor_SMD:R_0603_1608Metric, symbol Device:R_US
- added U1: TPD4E05U06DQA, Package_SON:USON-10_2.5x1.0mm_P0.5mm, symbol Power_Protection:TPD4E05U06DQA
- J1: footprint Connector_Molex:Molex_Micro-Fit_3.0_43045-1212_2x06_P3.00mm_Vertical -> Connector_Molex:Molex_Micro-Fit_3.0_43045-1200_2x06_P3.00mm_Horizontal
- Q3: value AO3401A -> AO3407A
- R1: value R -> 13k
- R22: value 330 -> 47
- R7: value 12k -> 100k
- R9: value 3k -> 47
Connections:
- net +3.3V: now also R4.2; no longer R4.1
- net BAT+: now also J1.1 (Pin_1); no longer J1.12 (Pin_12)
- net BMS Fault: now also J1.8 (Pin_8), R4.1, U5.9 (PA2), U1.4 (D2+); no longer J1.5 (Pin_5), R9.2
- net BSPD Fault: now also D8.1 (A1), J1.12 (Pin_12); no longer J1.1 (Pin_1)
- net BSPD_gate: no longer D8.1 (A1)
- net Extra_GPIO1: now also J1.5 (Pin_5); no longer J1.11 (Pin_11)
- net Extra_GPIO2: now also J1.4 (Pin_4); no longer J1.9 (Pin_9)
- net GND: now also R27.1, U1.3 (GND), U1.8 (GND)
- net IMD Fault: now also D8.2 (A1), J1.6 (Pin_6); no longer J1.3 (Pin_3)
- net IMD_Gate: no longer D8.2 (A1)
- net No_Faults: now also J1.7 (Pin_7), U5.17 (PA10/PA12), U1.5 (D2-); no longer J1.10 (Pin_10)
- net Precharge_fault: now also J1.3 (Pin_3); no longer J1.6 (Pin_6)
- net Reset: now also J1.9 (Pin_9), R14.1, U5.8 (PA1), U1.1 (D1+); no longer J1.4 (Pin_4), R22.1
- net Reset_Latch: now also R22.1, U5.3 (PC15); no longer Q3.1 (G), U5.10 (PA3)
- net SDC 1: now also J1.11 (Pin_11); no longer J1.8 (Pin_8)
- net SDC 2: now also J1.10 (Pin_10); no longer J1.7 (Pin_7)
- net at Q2.3 (D), R19.2: now also U5.2 (PC14); no longer U5.8 (PA1)
- net BMS_Gate: now reaches U5.1 (PB7)
- net BMS_Gate: now also R9.2
- net at U5.11 (PA4): now also R15.1
- net +12V renamed GLV+
- net GLV+: now also R26.2
- net BMS_gate: no longer names the net of Q10.1 (G), R7.2, R9.1
- net BMS_gate: no longer Q4.1 (G)
- net Precharge_gate: no longer names the net of Q11.1 (G), R13.1, R16.2
- new net: Q4.1 (G), R22.2, R27.2
- new net: Q4.3 (D), R25.1
- new net: Q3.1 (G), R25.2, R26.1
- now unconnected: U5.15 (PA8)
- no-connect marks 14 -> 13
Other:
- note added: "BMS_fault is the discharge enable pin (open drain), pulled low when active (safe to discharge), floating when not on (fault)"
- note removed: "Fix VDD Decoupling capacitors according to datasheet of https://www.st.com/resource/en/datasheet/stm32c011f4.pdf"
- note removed: "For ESD protection"
- moved on the sheet: 3V1, C1, C2, C6, C7, D1, D10, D11, D13, D14, D15, D16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

Commit message: updated relayboard
Parts:
- removed Q7: AO3400A, Package_TO_SOT_SMD:SOT-23, symbol Transistor_FET:AO3400A
- removed R23: 100k, Resistor_SMD:R_0603_1608Metric, symbol Device:R_US
- removed R24: 47, Resistor_SMD:R_0603_1608Metric, symbol Device:R_US
- removed U1: TPD4E05U06DQA, Package_SON:USON-10_2.5x1.0mm_P0.5mm, symbol Power_Protection:TPD4E05U06DQA
- added D7: SD15_SOD323, Diode_SMD:D_SOD-323, symbol Diode:SD15_SOD323
- added Q12: AO3407A, Package_TO_SOT_SMD:SOT-23, symbol Transistor_FET:AO3401A
- added Q8: AO3400A, Package_TO_SOT_SMD:SOT-23, symbol Transistor_FET:AO3400A
- added R28, R31: 100k, Resistor_SMD:R_0603_1608Metric, symbol Device:R_US
- added R29, R30: 47, Resistor_SMD:R_0603_1608Metric, symbol Device:R_US
- added R3: 100, Resistor_SMD:R_0603_1608Metric, symbol Device:R_US
- added U2: TPD4E05U06DQA, Package_SON:USON-10_2.5x1.0mm_P0.5mm, symbol Power_Protection:TPD4E05U06DQA
- C1: value 10μF -> 0.33μF
- C2: value 22μF -> 0.1μF
- D17: footprint Diode_SMD:D_SOD-123F -> Diode_SMD:D_SOD-323
- D8: value PSM712-LF-T7 -> AZ23C10
- J2: footprint Connector_PinHeader_2.54mm:PinHeader_1x04_P2.54mm_Vertical_SMD_Pin1Left -> Connector_PinHeader_2.54mm:PinHeader_1x04_P2.54mm_Vertical
- R10, R11, R12, R6: value 4.7K -> 10k
- R17, R5: value 3k -> 12k
Connections:
- net BAT+: now also D7.1 (A1)
- net BMS Fault: now also U2.4 (D2+)
- net BSPD Fault: no longer D8.1 (A1)
- net BSPD_gate: now also D8.1 (A1)
- net GLV+: now also Q12.2 (S), R31.2
- net GND: now also D7.2 (A2), Q8.2 (S), R28.1, U2.3 (GND), U2.8 (GND)
- net IMD Fault: no longer D8.2 (A1)
- net IMD_Gate: now also D8.2 (A1)
- net No_Faults: now also R3.2, U2.5 (D2-); no longer U5.17 (PA10/PA12)
- net Precharge_fault: now also U2.2 (D1-)
- net Reset: now also U2.1 (D1+)
- net at U5.16 (PA9/PA11): now also R29.1
- net Extra_GPIO1 renamed Extra_GPIO_LOW
- net Extra_GPIO2 renamed Extra_GPIO_High
- net Extra_GPIO_High: now also Q12.3 (D)
- new net: R3.1, U5.17 (PA10/PA12)
- new net: Q8.1 (G), R28.2, R29.2
- new net: Q8.3 (D), R30.1
- new net: Q12.1 (G), R30.2, R31.1
Other:
- note added: "Active Low fault"
- note added: "No Faults is Push/Pull Output to Roll Hoop MCU (series resistor for short protection)"
- note removed: "No Faults is Active High Output to Roll Hoop MCU (series resistor for protection)"

Commit message: Relayboard fixes
Parts:
- removed Q2: AO3400A, Package_TO_SOT_SMD:SOT-23, symbol Transistor_FET:AO3400A
- added R23: 8.3k, Resistor_SMD:R_0603_1608Metric, symbol Device:R_US
- R17: value 12k -> 47
- R19: value 10k -> 27k
Connections:
- net +3.3V: no longer R19.1
- net GND: now also R23.2
- net IMD Fault: now also R19.1; no longer R17.2
- net IMD_Gate: no longer Q9.1 (G), R17.1, R18.2
- net at R19.2: now also U5.13 (PA6), R23.1; no longer U5.2 (PC14)
- net IMD GATE: now reaches U5.7 (PA0)
- net IMD GATE: now also R17.2
- new net: Q9.1 (G), R17.1, R18.2
Other:
- moved on the sheet: C6, R14, R15, R17, R18, R3, R4, U5

Commit message: relayboard fixes
Connections:
- net IMD_Gate: now also R17.2, U5.20 (PB6)
- net IMD GATE: no longer names the net of U5.7 (PA0)
- net IMD GATE: no longer R17.2
Changed lines of the file:
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@@
 		)
 	)
-	(global_label "IMD GATE"
+	(global_label "IMD_Gate"
 		(shape input)
 		(at 69.85 158.75 270)
@@
 		)
 		(property "Intersheetrefs" "${INTERSHEET_REFS}"
-			(at 69.85 170.5042 90)
+			(at 69.85 170.2623 90)
 			(effects
 				(font
@@
 		)
 	)
+	(global_label "IMD_Gate"
+		(shape input)
+		(at 271.78 165.1 180)
+		(fields_autoplaced yes)
+		(effects
+			(font
+				(size 1.27 1.27)
+			)
+			(justify right)
+		)
+		(property "Intersheetrefs" "${INTERSHEET_REFS}"
+			(at 260.2677 165.1 0)
+			(effects
+				(font
+					(size 1.27 1.27)
+				)
+				(justify right)
+				(hide yes)
+			)
+		)
+	)
 	(global_label "GLV+"
 		(shape input)
@@
 				(hide yes)
 			)
-		)
-	)
-	(global_label "IMD GATE"
-		(shape input)
-		(at 307.34 152.4 0)
-		(fields_autoplaced yes)
-		(effects
-			(font
-				(size 1.27 1.27)
-			)
-			(justify left)
-		)
-		(property "Intersheetrefs" "${INTERSHEET_REFS}"
-			(at 319.0942 152.4 0)
-			(effects
-				(font
-					(size 1.27 1.27)
-				)
-				(justify left)
-				(hide yes)
-			)
