File: 2025-26/Boards/RML/RML_V2/RML-26_V2.kicad_pcb (KiCad board)
At the start: 2 copper layers, 90.1 x 30 mm, 26 parts, among them J1 043045-0412, Q2 AO3401A, Q3 UJ3N065080K3S, Q4 AO3401A, U1 H11L1M, U2 NE555D

Commit message: RML_V2
Parts:
- added HV-: 043045-0212, Connector_Molex:Molex_Micro-Fit_3.0_43045-0212_2x01_P3.00mm_Vertical, F.Cu at (117.5, 82.6)
- moved HV+ 12.2 mm to (117.5, 98.5)
- moved F1 8.74 mm to (108.8, 93.2), turned to 0 degrees
- moved F2 8.68 mm to (108.8, 87.7), turned to 180 degrees
- moved D4 4.52 mm to (124.7, 77.5)
- moved R6 4.41 mm to (128.4, 77.4)
- moved D1 3.34 mm to (123.5, 79.8)
- moved Q3 2.04 mm to (124.5, 84.3)
- moved D3 1.77 mm to (118.2, 91.2)
- moved G*** 0.64 mm to (151.5, 101.1)
- renumbered Molex1 to HV+
Connections:
- F2 pad 2: Net-(Molex1-Pin_1) -> Net-(Molex2-Pin_1)
- HV+ pad 1: Net-(Molex1-Pin_1) -> /HV+
- HV+ pad 2: /HV+ -> unconnected-(Molex1-Pin_2-Pad2)
Routing:
- net Net-(R6-Pad2): track 16.9 -> 41.7 mm
- net Net-(Molex2-Pin_1): track 0.00 -> 13.3 mm
- net Net-(D3-K): track 1.87 -> 7.23 mm
- net /HV-: track 68.9 -> 74.2 mm
- net Net-(D1-K): track 19.7 -> 24.9 mm
- net /HV+: track 10.9 -> 13.5 mm
- net Net-(D3-A): track 4.98 -> 6.35 mm
- added copper zone on F.Cu, net Net-(D3-A)
- removed copper zone on F.Cu, net Light+
