File: 2025-26/Boards/RML/RML_V2/RML-26_V2.kicad_sch (KiCad schematic)
At the start: 25 parts, among them J1 043045-0412, Q2 AO3401A, Q3 UJ3N065080K3S, Q4 AO3401A, U1 H11L1M, U2 NE555D

Commit message: RML_V2
Parts:
- added Molex2: 043045-0212, Connector_Molex:Molex_Micro-Fit_3.0_43045-0212_2x01_P3.00mm_Vertical, symbol Connector_Generic:Conn_01x02
Connections:
- net HV+: now also Molex1.1 (Pin_1); no longer Molex1.2 (Pin_2)
- net at F2.2: now also Molex2.1 (Pin_1); no longer Molex1.1 (Pin_1)
Other:
- moved on the sheet: Molex1
Changed lines of the file:
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@@
+	(wire
+		(pts
+			(xy 36.83 52.07) (xy 36.83 75.565)
+		)
+		(stroke
+			(width 0)
+			(type default)
+		)
+	)
 	(wire
 		(pts
@@
 	(wire
 		(pts
-			(xy 36.83 52.07) (xy 36.83 80.01)
-		)
-		(stroke
-			(width 0)
-			(type default)
-		)
-	)
-	(wire
-		(pts
 			(xy 157.48 38.1) (xy 157.48 41.91)
 		)
@@
 	(wire
 		(pts
+			(xy 36.83 85.09) (xy 36.83 90.17)
+		)
+		(stroke
+			(width 0)
+			(type default)
+		)
+	)
+	(wire
+		(pts
 			(xy 170.18 80.01) (xy 170.18 81.28)
 		)
@@
 	(wire
 		(pts
+			(xy 35.56 75.565) (xy 36.83 75.565)
+		)
+		(stroke
+			(width 0)
+			(type default)
+		)
+	)
+	(wire
+		(pts
 			(xy 86.36 68.58) (xy 102.87 68.58)
 		)
@@
 		(pts
 			(xy 146.05 77.47) (xy 143.51 77.47)
-		)
-		(stroke
-			(width 0)
-			(type default)
-		)
-	)
-	(wire
-		(pts
-			(xy 36.83 82.55) (xy 36.83 90.17)
 		)
 		(stroke
@@
 	)
 	(symbol
+		(lib_id "Connector_Generic:Conn_01x02")
+		(at 31.75 85.09 180)
+		(unit 1)
+		(exclude_from_sim no)
+		(in_bom yes)
+		(on_board yes)
+		(dnp no)
+		(property "Reference" "Molex2"
+			(at 22.225 82.55 0)
+			(effects
+				(font
+					(size 1.27 1.27)
+				)
+			)
+		)
+		(property "Value" "043045-0212"
+			(at 22.225 85.09 0)
+			(effects
+				(font
+					(size 1.27 1.27)
+				)
+			)
+		)
+		(property "Footprint" "Connector_Molex:Molex_Micro-Fit_3.0_43045-0212_2x01_P3.00mm_Vertical"
+			(at 31.75 85.09 0)
+			(effects
+				(font
+					(size 1.27 1.27)
+				)
+				(hide yes)
+			)
+		)
+		(property "Datasheet" "~"
+			(at 31.75 85.09 0)
+			(effects
+				(font
+					(size 1.27 1.27)
+				)
+				(hide yes)
+			)
+		)
+		(property "Description" ""
+			(at 31.75 85.09 0)
+			(effects
+				(font
+					(size 1.27 1.27)
+				)
+				(hide yes)
+			)
+		)
+		(pin "1"
+		)
+		(pin "2"
+		)
+		(instances
+			(project "RML-26_V2"
+				(path "/d0262e13-a8ab-42db-962e-1ef7dd9c8d4a"
+					(reference "Molex2")
+					(unit 1)
+				)
+			)
+		)
+	)
+	(symbol
 		(lib_id "Device:Fuse")
 		(at 36.83 93.98 180)
@@
 		)
 		(property "Value" "043045-0412"
-			(at 111.76 30.48 0)
+			(at 120.65 30.48 0)
 			(effects
 				(font
@@
 	(symbol
 		(lib_id "Connector_Generic:Conn_01x02")
-		(at 31.75 82.55 180)
+		(at 30.48 75.565 180)
 		(unit 1)
 		(exclude_from_sim no)
@@
 		(dnp no)
 		(property "Reference" "Molex1"
-			(at 22.225 80.01 0)
+			(at 20.955 73.025 0)
 			(effects
 				(font
@@
 		)
 		(property "Value" "043045-0212"
-			(at 22.225 82.55 0)
+			(at 20.955 75.565 0)
 			(effects
 				(font
@@
 		)
 		(property "Footprint" "Connector_Molex:Molex_Micro-Fit_3.0_43045-0212_2x01_P3.00mm_Vertical"
-			(at 31.75 82.55 0)
+			(at 30.48 75.565 0)
 			(effects
 				(font
@@
 		)
 		(property "Datasheet" "~"
-			(at 31.75 82.55 0)
+			(at 30.48 75.565 0)
 			(effects
 				(font
@@
 		)
 		(property "Description" ""
-			(at 31.75 82.55 0)
-			(effects
-				(font
+			(at 30.48 75.565 0)
+			(effects
+				(font
