File: 2025-26/Boards/Rollhoop_Board/Rollhoop_Simple/Rollhoop_Simple/Roll_Hoop_Board.kicad_sch (KiCad schematic)
At the start: 7 parts, among them J1 DTM13-12PA, J2 DTM13-12PA

Commit message: adding updated rollhoop board
Parts:
- removed Back_Panel1: 043045-0212, Connector_Molex:Molex_Micro-Fit_3.0_43045-0212_2x01_P3.00mm_Vertical, symbol Connector_Generic:Conn_01x02
- added J5: 043045-0612, Connector_Molex:Molex_Micro-Fit_3.0_43045-0612_2x03_P3.00mm_Vertical, symbol Connector_Generic:Conn_01x06
- added SW1, SW2: 84-5330.0020, symbol Switch:SW_SPST
- J4: renamed from Front_Panel1; footprint (none) -> Connector_Molex:Molex_Micro-Fit_3.0_43045-0612_2x03_P3.00mm_Vertical
Connections:
- net +12V: now also J5.5 (Pin_5), J5.6 (Pin_6); no longer J1.5, J2.5, J4.4 (Pin_4)
- net CAN_H: now also J2.2; no longer J2.7
- net CAN_L: now also J2.1; no longer J2.6
- net CAN_S: now also J2.12; no longer J2.8
- net DSH_SDC_IN: now also J2.10, SW2.1 (A); no longer J2.2
- net GND: now also J2.6, J4.1 (Pin_1), J5.1 (Pin_1); no longer J2.11
- net Green_Out: now also J2.8, J4.2 (Pin_2), J5.2 (Pin_2); no longer J2.3, J4.1 (Pin_1)
- net RLH_RML_YELLOW: now also J4.4 (Pin_4), J5.4 (Pin_4); no longer J4.3 (Pin_3)
- net RLH_SDC_IN: now also E-Stops1.2 (Pin_2), SW1.2 (B)
- net Red_Out: now also J2.5, J4.3 (Pin_3), J5.3 (Pin_3); no longer J2.4, J4.2 (Pin_2)
- net Speaker_Out: now also J2.7; no longer J2.10
- net Extra: now reaches J1.10
- net DSH_PWR: now reaches J1.4
- net DSH_PWR: now also J2.11
- net RLH_SDC_OUT renamed DSH_SDC_OUT
- net DSH_SDC_OUT: no longer E-Stops1.2 (Pin_2)
- new net: SW1.1 (A), SW2.2 (B)
- new net RLH_PWR: J1.5
Other:
- note added: "CAN Transceiver and STM32"
- note added: "SDC goes out to Switches then back into board"
- note added: "Shutdown Circuit"
- moved on the sheet: E-Stops1, J1, J4, Speaker1, Speaker2
