File: 2026-27/Boards/VCU/VCU/VCU.kicad_sch (KiCad schematic)
At the start: 37 parts, among them J1 5810148005, J2 Conn_01x02_Socket, J3 Conn_01x04_Socket, J4 TC2030, U1 STM32F405VGTx, U3 ESP32-WROOM-32E, X1 X49SM8MSD2SC

Commit message: Analog/Digital Inputs Added
Parts:
- added C21, C22, C28, C29, C30: 100nF, PCM_JLCPCB:C_0603, symbol PCM_JLCPCB-Capacitors:0603,100nF
- added C23: 4.7uF, PCM_JLCPCB:C_0603, symbol PCM_JLCPCB-Capacitors:0603,4.7uF
- added C24, C41: 100pF, PCM_JLCPCB:C_0805, symbol PCM_JLCPCB-Capacitors:0805,100pF
- added C25, C26: 0603B472K500NT, PCM_JLCPCB:C_0603, symbol JLCImport:0603B472K500NT
- added C27, C31: CL21A106KAYNNNE, PCM_JLCPCB:C_0805, symbol JLCImport:CL21A106KAYNNNE
- added C32: GRM1885C1H103JA01D, PCM_JLCPCB:C_0603, symbol JLCImport:GRM1885C1H103JA01D
- added C35: 10uF, PCM_JLCPCB:C_0805, symbol PCM_JLCPCB-Capacitors:0805,10uF
- added C40: VZH221M1CTR-0607, easyeda2kicad:CAP-SMD_BD6.3-L6.6-W6.6-RD, symbol button:VZH221M1CTR-0607
- added C42: 2.2uF, PCM_JLCPCB:C_0805, symbol PCM_JLCPCB-Capacitors:0805,2.2uF
- added C46: 10nF, PCM_JLCPCB:C_0805, symbol PCM_JLCPCB-Capacitors:0805,10nF
- added C47, C48, C55: 10uF, PCM_JLCPCB:C_0805, symbol PCM_JLCPCB-Capacitors:0805,10uF,(2)
- added D1: SMAJ26CA, Diode_SMD:D_SMA, symbol Diode:SMAJ26CA
- added D2, D3: ESD2CANFD24DBZR, Package_TO_SOT_SMD:SOT-23-3, symbol JLCImport:ESD2CANFD24DBZR
- added D4: SS54, PCM_JLCPCB:D_SMA, symbol PCM_JLCPCB-Diodes:Schottky,SS54
- added D5: BAV199_215, Package_TO_SOT_SMD:SOT-23-3, symbol JLCImport:BAV199_215
- added DC1: DC-012A-B200, easyeda2kicad:DC-IN-TH_DC-012A-B200, symbol easyeda2kicad:DC-012A-B200
- added F1: Fuse, Fuse:Fuse_0805_2012Metric, symbol Device:Fuse
- added J5: 472192001, micro-sd:CONN_47219-2001_MOL, symbol sdcardconnector:472192001
- added J7: USB_OTG, Connector_USB:USB_Micro-AB_Molex_47590-0001, symbol Connector:USB_OTG
- added L2: CYH127-15UH, easyeda2kicad:IND-SMD_L12.3-W12.3, symbol button:CYH127-15UH
- added L4, L5: ACT1210-101-2P-TL00, PCM_JLCPCB:OSC-SMD_4P-L3.2-W2.5-BL, symbol JLCImport:ACT1210-101-2P-TL00
- added Q6: AOD4184A, AOD4184A:DPAK228P994X240-4N, symbol mosfet-rp:AOD4184A
- added R10, R7, R8, R9: AC0805FR-0760R4L, PCM_JLCPCB:R_0805, symbol JLCImport:AC0805FR-0760R4L
- added R11, R17: 10k, Resistor_SMD:R_0201_0603Metric, symbol Device:R
- added R12, R14, R15, R16: 1206W4F1001T5E, PCM_JLCPCB:R_1206, symbol JLCImport:1206W4F1001T5E
- added R13: FRC1206F4700TS, PCM_JLCPCB:R_1206, symbol JLCImport:FRC1206F4700TS
- added R18: 0805W8F4701T5E, PCM_JLCPCB:R_0805, symbol JLCImport:0805W8F4701T5E
- added R19: 0805W8F6801T5E, PCM_JLCPCB:R_0805, symbol JLCImport:0805W8F6801T5E
- added R51, R52, R54, R55, R67: 47kΩ, PCM_JLCPCB:R_0603, symbol PCM_JLCPCB-Resistors:0603,47kΩ
- added R53: 4.7kΩ, PCM_JLCPCB:R_0603, symbol PCM_JLCPCB-Resistors:0603,4.7kΩ
- added R57, R70: 10kΩ, PCM_JLCPCB:R_0603, symbol PCM_JLCPCB-Resistors:0603,10kΩ
- added R71: 0603WAF3241T5E, easyeda2kicad:R0603, symbol button:0603WAF3241T5E
- added U2: LSM6DS3, Package_LGA:LGA-14_3x2.5mm_P0.5mm_LayoutBorder3x4y, symbol Sensor_Motion:LSM6DS3
- added U20: LDL1117S33R, easyeda2kicad:SOT-223-4_L6.5-W3.5-P2.30-LS7.0-BR, symbol button:LDL1117S33R
- added U23: USBLC6-4SC6, Package_TO_SOT_SMD:SOT-23-6, symbol Power_Protection:USBLC6-4SC6
- added U25: LM74610QDGKRQ1, symbol reverse-polarity-protection:LM74610QDGKRQ1
- added U26, U27: SN65HVD230DR, PCM_JLCPCB:SOIC-8_L4.9-W3.9-P1.27-LS6.0-BL, symbol PCM_JLCPCB-Interface:Transceiver, CAN, SN65HVD230DR
- added U28: TPS5430DDA, Package_SO:TI_SO-PowerPAD-8_ThermalVias, symbol Regulator_Switching:TPS5430DDA
- added U29, U30, U31: RH-5000, easyeda2kicad:TEST-TH_BD2.54-P1.4_RED, symbol easyeda2kicad:RH-5000
- added U4, U5: LTV-357T-C_C119091, PCM_JLCPCB:MBS_L4.7-W3.8-P2.40-LS7.0-TL, symbol JLCImport:LTV-357T-C_C119091
Connections:
- net +3.3V: now also C21.2, C22.2, C27.2, C28.2, C29.2, C30.1, C31.2, C35.2, C55.1, D5.2, R11.2, R17.2, R51.2, R52.2, R54.2, R55.1, R67.1, U2.5 (VDDIO), U2.8 (VDD), U20.4 (VOUT), U26.3 (VCC), U27.3 (VCC)
- net GND: now also C21.1, C22.1, C23.1, C24.2, C25.1, C26.1, C27.1, C28.1, C29.1, C30.2, C31.1, C32.1, C35.1, C40.2, C41.2, C47.1, C48.1, C55.2, D1.1 (A1), D2.3 (GND), D3.3 (GND), D4.2, D5.1, DC1.2, J7.5 (GND), J7.6 (Shield), R19.2, R57.2, R71.1, U2.6 (GND), U2.7 (GND), U20.1 (GND), U23.2 (GND), U23.3 (I/O2), U26.2 (GND), U26.8 (RS), U27.2 (GND), U27.8 (RS), U28.6 (GND), U28.9 (GNDPAD), U31.1, U4.2, U4.3, U5.2, U5.3
- net CAN1+: now reaches J1.10
- net CAN1+: now also D2.2 (IO), L4.4
- net CAN1-: now reaches J1.15
- net CAN1-: now also D2.1 (IO), L4.3
- net CAN0-: now reaches J1.8
- net CAN0-: now also D3.1 (IO), L5.3
- net CAN0+: now reaches J1.9
- net CAN0+: now also D3.2 (IO), L5.4
- new net: C24.1, D1.2 (A2), F1.1, Q6.3, U25.4 (ANODE)
- new net: R70.2, R71.2, U28.4 (VSENSE)
- new net: L5.1, R9.2, U27.7 (CANH)
- new net: R12.2, U4.1
- new net: R14.1, U4.4
- new net: R13.2, U5.1
- new net: L4.1, R8.2, U26.7 (CANH)
- new net: L4.2, R7.1, U26.6 (CANL)
- new net: L5.2, R10.1, U27.6 (CANL)
- new net: D5.3, R16.2, R18.2, R19.1
- new net: R15.1, U5.4
- new net: C23.2, J7.1 (VBUS), R53.1, U23.5 (VBUS)
- new net: C46.1, U28.1 (BOOT)
- new net: C46.2, D4.1, L2.1, U28.8 (PH)
- new net: C42.1, U25.7 (VCAPH)
- new net: C42.2, U25.1 (VCAPL)
- new net: Q6.1, U25.2 (GATE_PULL_DOWN), U25.6 (GATE_DRIVE)
- new net +12V: C41.1, C48.2, DC1.1, Q6.4, U25.8 (CATHODE), U28.7 (VIN), U29.1
- new net +5V: C40.1, C47.2, L2.2, R70.1, U20.3 (VIN), U30.1
- new net 12VDIN: R12.1
- new net 12VGPIO: R11.1, R14.2
- new net 2Vref: C26.2, R10.2, R9.1, U27.5 (VREF)
- new net 5VAIN: R18.1
- new net 5VDIN: R13.1
- new net 5VGPIO: R15.2, R17.1
- new net AIO: C32.2, R16.1
- new net CAN0RX: U27.4 (R)
- new net CAN0TX: U27.1 (D)
- new net CAN1RX: U26.4 (R)
- new net CAN1TX: U26.1 (D)
- new net EX 12V: F1.2
- new net PA10 (ID): J7.4 (ID), U23.4 (I/O3)
- new net PA11 (D-): J7.2 (D-), U23.6 (I/O4)
- new net PA12 (D+): J7.3 (D+), U23.1 (I/O1)
- new net PA9 (VBUS): R53.2, R57.1
- new net PB0 (MPU_INT): U2.4 (INT1)
- new net PB12 (MPU_CS_N): U2.12 (CS)
- new net PB13 (MPU_SCLK): U2.3 (SCX)
- new net PB14 (MISO): U2.1 (SDO/SA0)
- new net PB15 (MOSI): U2.2 (SDX)
- new net PC10 (DAT2): R51.1
- new net PC11 (CD/DAT3): R52.1
- new net PC8 (DAT0): R55.2
- new net PC9 (DAT1): R67.2
- new net PD2 (CMD): R54.1
- new net Vref: C25.2, R7.2, R8.1, U26.5 (VREF)
- no-connect marks 0 -> 5
Other:
- note added: "1. External 12V Power comes in"
- note added: "12-5V 2A buck converter"
- note added: "12V Buck ~ 1.6A 4 12V Outputs ~ 4 x 100mA 2A, upsize to 5A for temp headroom"
- note added: "12V Power"
- note added: "2. Passes through protection IC, outputs to 12V flag"
- note added: "3. Converts to 5V"
- note added: "4. Converts to 3.3V from 5V"
- note added: "4.5A 15uH ±20% 28.6mΩ"
- note added: "500mA"
- note added: "5V-3.3V, 1.2A, MaxVin 18V"
- note added: "Analog Inputs"
- note added: "CAN Transceiver w/ ESD"
- note added: "Digital Inputs"
- note added: "EN can be left floating"
- note added: "ESP32 OTA PROG"
- note added: "I oversized capacitor to account for any capacitance loss due to ceramic"
- note added: "Low active SPI"
- note added: "MPU 6 axis, accel + gyro w/fifo"
- note added: "Micro-SD CARD"
- note added: "Reverse Polarity Protection"
- note added: "USB OTG + ESD Protection"
- note added: "input can be (5.5v to 36V)"
- note added: "pull up resistors for data lines (47k)"
- moved on the sheet: J1

Commit message: Finished schematic
Parts:
- removed C21, C22, C30: 100nF, PCM_JLCPCB:C_0603, symbol PCM_JLCPCB-Capacitors:0603,100nF
- removed C23: 4.7uF, PCM_JLCPCB:C_0603, symbol PCM_JLCPCB-Capacitors:0603,4.7uF
- removed C24, C41: 100pF, PCM_JLCPCB:C_0805, symbol PCM_JLCPCB-Capacitors:0805,100pF
- removed C32: GRM1885C1H103JA01D, PCM_JLCPCB:C_0603, symbol JLCImport:GRM1885C1H103JA01D
- removed C35: 10uF, PCM_JLCPCB:C_0805, symbol PCM_JLCPCB-Capacitors:0805,10uF
- removed C42: 2.2uF, PCM_JLCPCB:C_0805, symbol PCM_JLCPCB-Capacitors:0805,2.2uF
- removed C47, C55: 10uF, PCM_JLCPCB:C_0805, symbol PCM_JLCPCB-Capacitors:0805,10uF,(2)
- removed D1: SMAJ26CA, Diode_SMD:D_SMA, symbol Diode:SMAJ26CA
- removed D5: BAV199_215, Package_TO_SOT_SMD:SOT-23-3, symbol JLCImport:BAV199_215
- removed DC1: DC-012A-B200, easyeda2kicad:DC-IN-TH_DC-012A-B200, symbol easyeda2kicad:DC-012A-B200
- removed F1: Fuse, Fuse:Fuse_0805_2012Metric, symbol Device:Fuse
- removed J3: Conn_01x04_Socket, symbol Connector:Conn_01x04_Socket
- removed J5: 472192001, micro-sd:CONN_47219-2001_MOL, symbol sdcardconnector:472192001
- removed Q6: AOD4184A, AOD4184A:DPAK228P994X240-4N, symbol mosfet-rp:AOD4184A
- removed R13: FRC1206F4700TS, PCM_JLCPCB:R_1206, symbol JLCImport:FRC1206F4700TS
- removed R15, R16: 1206W4F1001T5E, PCM_JLCPCB:R_1206, symbol JLCImport:1206W4F1001T5E
- removed R17: 10k, Resistor_SMD:R_0201_0603Metric, symbol Device:R
- removed R18: 0805W8F4701T5E, PCM_JLCPCB:R_0805, symbol JLCImport:0805W8F4701T5E
- removed R19: 0805W8F6801T5E, PCM_JLCPCB:R_0805, symbol JLCImport:0805W8F6801T5E
- removed R51, R52, R54, R55, R67: 47kΩ, PCM_JLCPCB:R_0603, symbol PCM_JLCPCB-Resistors:0603,47kΩ
- removed R53: 4.7kΩ, PCM_JLCPCB:R_0603, symbol PCM_JLCPCB-Resistors:0603,4.7kΩ
- removed R57, R70: 10kΩ, PCM_JLCPCB:R_0603, symbol PCM_JLCPCB-Resistors:0603,10kΩ
- removed U2: LSM6DS3, Package_LGA:LGA-14_3x2.5mm_P0.5mm_LayoutBorder3x4y, symbol Sensor_Motion:LSM6DS3
- removed U25: LM74610QDGKRQ1, symbol reverse-polarity-protection:LM74610QDGKRQ1
- removed U31: RH-5000, easyeda2kicad:TEST-TH_BD2.54-P1.4_RED, symbol easyeda2kicad:RH-5000
- removed U5: LTV-357T-C_C119091, PCM_JLCPCB:MBS_L4.7-W3.8-P2.40-LS7.0-TL, symbol JLCImport:LTV-357T-C_C119091
- added C21, C30: GRM188Z71C475KE21D, Capacitor_SMD:C_0603_1608Metric, symbol JLCImport:GRM188Z71C475KE21D
- added C22, C23, C24, C33, C34, C35: 100nF, Capacitor_SMD:C_0402_1005Metric, symbol Device:C
- added C36, C37, C38, C39, C41, C42, C43, C44, C45, C47, C53, C54: GRM1885C1H103JA01D, PCM_JLCPCB:C_0603, symbol JLCImport:GRM1885C1H103JA01D
- added C49, C50, C51, C52: 10uF, PCM_JLCPCB:C_0805, symbol PCM_JLCPCB-Capacitors:0805,10uF,(2)
- added CN1: 436500200, Connector_Molex:Molex_Micro-Fit_3.0_43045-0212_2x01_P3.00mm_Vertical, symbol JLCImport:436500200
- added Card1: DM3AT-SF-PEJM5, Crystal:Crystal_SMD_HC49-SD, symbol JLCImport:DM3AT-SF-PEJM5
- added D1: BZT52C15, Diode_SMD:D_SOD-123, symbol JLCImport:BZT52C15
- added D10, D11, D12, D13, D14, D15, D16, D17, D18, D19, D8, D9: BAV199_215, Package_TO_SOT_SMD:SOT-23-3, symbol JLCImport:BAV199_215
- added D6: TPD6E004RSER, Package_DFN_QFN:ST_UQFN-6L_1.5x1.7mm_P0.5mm, symbol JLCImport:TPD6E004RSER
- added D7: SMAJ18A_C148219, Package_SO:SOP-4_4.4x2.6mm_P1.27mm, symbol JLCImport:SMAJ18A_C148219
- added H1, H2, H3: PZ254V-11-04P_C2691448, TerminalBlock:TerminalBlock_Xinya_XY308-2.54-4P_1x04_P2.54mm_Horizontal, symbol JLCImport:PZ254V-11-04P_C2691448
- added LED1: KT-0603R, LED_SMD:LED_LiteOn_LTST-C295K_1.6x0.8mm, symbol JLCImport:KT-0603R
- added Q1: IRFR9024N_C2874613, Package_TO_SOT_THT:TO-5-3, symbol JLCImport:IRFR9024N_C2874613
- added Q2, Q3, Q4, Q5, Q6, Q7, Q8, Q9: AO3400A, Package_TO_SOT_SMD:SOT-23-3, symbol JLCImport:AO3400A
- added R100, R104, R107, R110, R21: 0603WAF1003T5E, Resistor_SMD:R_0603_1608Metric, symbol JLCImport:0603WAF1003T5E
- added R101, R103, R106, R109, R13, R16, R19, R97: 0603WAF2200T5E, Resistor_SMD:R_0603_1608Metric, symbol JLCImport:0603WAF2200T5E
- added R102, R105, R111, R112, R113, R22, R23, R24, R25, R26, R27, R29, R32, R35, R38, R41, R50, R53, R56, R59: 10k, Resistor_SMD:R_0201_0603Metric, symbol Device:R
- added R108, R17, R30, R31, R33, R34, R36, R37, R39, R40, R42, R43, R44, R45, R46, R47, R49, R52, R55, R58, R64, R67, R70, R74, R77, R80, R83, R86, R89, R92, R95, R99: 1206W4F1001T5E, PCM_JLCPCB:R_1206, symbol JLCImport:1206W4F1001T5E
- added R15, R18, R96, R98: FRC0603F1003TS, Resistor_SMD:R_0603_1608Metric, symbol JLCImport:FRC0603F1003TS
- added R20: 0805W8F1000T5E, Resistor_SMD:R_0805_2012Metric, symbol JLCImport:0805W8F1000T5E
- added R28: 0603WAF1302T5E, Resistor_SMD:R_0603_1608Metric, symbol JLCImport:0603WAF1302T5E
- added R48, R51, R54, R57: FRC1206F4700TS, PCM_JLCPCB:R_1206, symbol JLCImport:FRC1206F4700TS
- added R60, R62, R65, R68, R72, R75, R78, R81, R84, R87, R90, R93: 0805W8F4701T5E, PCM_JLCPCB:R_0805, symbol JLCImport:0805W8F4701T5E
- added R61, R63, R66, R69, R73, R76, R79, R82, R85, R88, R91, R94: 0805W8F6801T5E, PCM_JLCPCB:R_0805, symbol JLCImport:0805W8F6801T5E
- added U10, U11, U12, U13, U14, U15, U16, U17, U18, U19, U9: LTV-357T-C_C119091, PCM_JLCPCB:MBS_L4.7-W3.8-P2.40-LS7.0-TL, symbol JLCImport:LTV-357T-C_C119091
- added U6: FRC0805F8661TS, Resistor_SMD:R_0805_2012Metric, symbol JLCImport:FRC0805F8661TS
- added U7: 0154002_DRT, Capacitor_THT:C_Rect_L10.3mm_W5.0mm_P7.50mm_MKS4, symbol JLCImport:0154002_DRT
- added U8: LSM6DS3TR-C, Package_LGA:Bosch_LGA-14_3x2.5mm_P0.5mm, symbol JLCImport:LSM6DS3TR-C
Connections:
- net 12VDIN is gone; now on net 12VDIN0: R12.1
- net BMSfault is gone; now on net 12VDIN1: J1.7
- net CAN0RX is gone; now on net CANRX2: U27.4 (R)
- net CAN0TX is gone; now on net CANTX2: U27.1 (D)
- net CAN1RX is gone; now on net CANRX1: U26.4 (R)
- net CAN1TX is gone; now on net CANTX1: U26.1 (D)
- net IMDfault is gone; now on net 12VDIN0: J1.6
- net TSMS is gone; now on net 12VDIN2: J1.1
- net Temp2 is gone; now on net 5VAIN7: J1.23
- net +12V: now also C49.2, D1.1 (K), D7.1, LED1.1 (A), Q1.3 (S), R102.2, R105.2, R108.2, R99.2
- net +3.3V: now also J1.21, U20.2 (VOUT), C22.2, C23.2, C30.2, C33.2, C34.2, C52.1, Card1.4 (VDD), D10.2, D11.2, D12.2, D13.2, D14.2, D15.2, D16.2, D17.2, D18.2, D19.2, D6.8 (VCC), D8.2, D9.2, H2.3, R111.2, R112.2, R113.2, R22.2, R23.2, R24.2, R25.1, R26.1, R29.2, R32.2, R35.2, R38.2, R41.2, R50.2, R53.2, R56.2, R59.2, U8.5 (VDDIO), U8.8 (VDD)
- net BOOT0: no longer R1.1, U1.94 (BOOT0)
- net EX 12V: now also J1.48, CN1.2, U7.1
- net GND: now also J1.17, J1.18, J1.22, J1.39, J1.46, J1.47, C21.2, C22.1, C23.1, C24.2, C30.1, C33.1, C34.1, C35.2, C36.1, C37.1, C38.1, C39.1, C41.1, C42.1, C43.1, C44.1, C45.1, C47.1, C49.1, C50.1, C51.1, C52.2, C53.1, C54.1, CN1.1, Card1.10, Card1.12, Card1.13, Card1.14, Card1.6 (VSS), Card1.9 (SW_B), D10.1, D11.1, D12.1, D13.1, D14.1, D15.1, D16.1, D17.1, D18.1, D19.1, D6.4 (GND), D7.2, D8.1, D9.1, H2.4, H3.4, Q2.2 (S), Q3.2 (S), Q4.2 (S), Q5.2 (S), R100.1, R104.1, R107.1, R110.1, R15.1, R18.1, R21.2, R27.1, R28.1, R61.2, R63.2, R66.2, R69.2, R73.2, R76.2, R79.2, R82.2, R85.2, R88.2, R91.2, R94.2, R96.1, R98.1, U10.2, U10.3, U11.2, U11.3, U12.2, U12.3, U13.2, U13.3, U14.2, U14.3, U15.2, U15.3, U16.2, U16.3, U17.2, U17.3, U18.2, U18.3, U19.2, U19.3, U8.2 (SDx), U8.3 (SCx), U8.6 (GND), U8.7 (GND), U9.2, U9.3; no longer U23.3 (I/O2)
- net PA11 (D-): now also U1.70 (PA11), U23.3 (I/O2); no longer U23.6 (I/O4)
- net PA12 (D+): now also U1.71 (PA12)
- net PA9 (VBUS): now also J7.1 (VBUS), U1.68 (PA9), U23.5 (VBUS), C35.1, R27.2
- net TCK: now also H1.3
- net TDI: now also H1.2
- net TDO: now also H1.4
- net TMS: now also H1.1
- net 5VDIN8: now reaches J1.11
- net 5VDIN8: now also R48.1
- net 5VDIN9: now reaches J1.12
- net 5VDIN9: now also R51.1
- net 12VDIN7: now reaches J1.16
- net 12VDIN7: now also U1.46 (PE15), R46.1
- net 5VAIN3: now reaches J1.19
- net 5VAIN3: now also R78.1
- net 12VDIN3: now reaches J1.2
- net 12VDIN3: now also U1.42 (PE11), R36.1
- net 5VAIN5: now reaches J1.29
- net 5VAIN5: now also R90.1
- net 12VDIN6: now reaches J1.3
- net 12VDIN6: now also U1.45 (PE14), R44.1
- net DOUT2: now reaches J1.31
- net DOUT2: now also Q4.3 (D)
- net DOUT3: now reaches J1.32
- net DOUT3: now also Q5.3 (D)
- net DOUT4: now reaches J1.33
- net DOUT4: now also Q6.3 (D), R102.1
- net 5VDIN11: now reaches J1.36
- net 5VDIN11: now also R57.1
- net 12VDIN5: now reaches J1.4
- net 12VDIN5: now also U1.44 (PE13), R42.1
- net DOUT5: now reaches J1.40
- net DOUT5: now also Q7.3 (D), R105.1
- net DOUT6: now reaches J1.41
- net DOUT6: now also Q8.3 (D), R99.1
- net DOUT7: now reaches J1.42
- net DOUT7: now also Q9.3 (D), R108.1
- net 5VDIN10: now reaches J1.43
- net 5VDIN10: now also R54.1
- net 12VDIN4: now reaches J1.5
- net 12VDIN4: now also U1.43 (PE12), R39.1
- net at R71.2, U28.4 (VSENSE): now also U6.1
- net STM-BOOT: now reaches U3.30 (IO18)
- net STM-BOOT: now also R1.1, U1.94 (BOOT0)
- net STM-NRST: now reaches U3.31 (IO19)
- net STM-NRST: now also C15.2, U1.14 (NRST), R20.2
- net GPIO_DOUT2: now reaches U1.1 (PE2)
- net GPIO_DOUT2: now also R19.1
- net AIO6: now reaches U1.15 (PC0)
- net AIO6: now also C36.2, R17.1
- net AIO7: now reaches U1.16 (PC1)
- net AIO7: now also C39.2, R70.1
- net AIO8: now reaches U1.17 (PC2)
- net AIO8: now also C42.2, R77.1
- net AIO9: now reaches U1.18 (PC3)
- net AIO9: now also C44.2, R83.1
- net GPIO_DOUT3: now reaches U1.2 (PE3)
- net GPIO_DOUT3: now also R97.1
- net AIO0: now reaches U1.23 (PA0)
- net AIO0: now also C37.2, R64.1
- net AIO1: now reaches U1.24 (PA1)
- net AIO1: now also C38.2, R67.1
- net AIO2: now reaches U1.25 (PA2)
- net AIO2: now also C41.2, R74.1
- net AIO3: now reaches U1.26 (PA3)
- net AIO3: now also C43.2, R80.1
- net AIO4: now reaches U1.29 (PA4)
- net AIO4: now also C45.2, R86.1
- net GPIO_DOUT4: now reaches U1.3 (PE4)
- net GPIO_DOUT4: now also R101.1
- net AIO5: now reaches U1.30 (PA5)
- net AIO5: now also C53.2, R92.1
- net SD_Detect: now reaches U1.32 (PA7)
- net SD_Detect: now also Card1.11 (SW_A)
- net AIO10: now reaches U1.33 (PC4)
- net AIO10: now also C47.2, R89.1
- net AIO11: now reaches U1.34 (PC5)
- net AIO11: now also C54.2, R95.1
- net IMU_SPI_INT_PB1: now reaches U1.36 (PB1)
- net IMU_SPI_INT_PB1: now also U8.4 (INT1)
- net GPIO_DOUT7: now reaches U1.38 (PE7)
- net GPIO_DOUT7: now also R109.1
- net 12VDIN0: now reaches U1.39 (PE8)
- net GPIO_DOUT5: now reaches U1.4 (PE5)
- net GPIO_DOUT5: now also R103.1
- net 12VDIN1: now reaches U1.40 (PE9)
- net 12VDIN1: now also R30.1
- net 12VDIN2: now reaches U1.41 (PE10)
- net 12VDIN2: now also R33.1
- net GPIO_DOUT6: now reaches U1.5 (PE6)
- net GPIO_DOUT6: now also R106.1
- net IMU_SPI_CS: now reaches U1.51 (PB12)
- net IMU_SPI_CS: now also R29.1, U8.12 (CS)
- net IMU_SPI_SCK: now reaches U1.52 (PB13)
- net IMU_SPI_SCK: now also U8.13 (SCL)
- net IMU_SPI_MISO: now reaches U1.53 (PB14)
- net IMU_SPI_MISO: now also U8.1 (SDO/SA0)
- net IMU_SPI_MOSI: now reaches U1.54 (PB15)
- net IMU_SPI_MOSI: now also U8.14 (SDA)
- net 5VGPIO8: now reaches U1.59 (PD12)
- net 5VGPIO8: now also R49.2, R50.1
- net 5VGPIO9: now reaches U1.60 (PD13)
- net 5VGPIO9: now also R52.2, R53.1
- net 5VGPIO10: now reaches U1.61 (PD14)
- net 5VGPIO10: now also R55.2, R56.1
- net 5VGPIO11: now reaches U1.62 (PD15)
- net 5VGPIO11: now also R58.2, R59.1
- net UART6_UTIL_TX: now reaches U1.63 (PC6)
- net UART6_UTIL_TX: now also H3.1
- net UART6_UTIL_RX: now reaches U1.64 (PC7)
- net UART6_UTIL_RX: now also H3.2
- net SD_D0: now reaches U1.65 (PC8)
- net SD_D0: now also Card1.7 (DAT0), D6.6 (IO5), R26.2
- net SD_D1: now reaches U1.66 (PC9)
- net SD_D1: now also Card1.8 (DAT1), D6.7 (IO6), R25.2
- net STM32_SWDIO: now reaches U1.72 (PA13)
- net STM32_SWDIO: now also H2.1
- net STM32_SWCLK: now reaches U1.76 (PA14)
- net STM32_SWCLK: now also H2.2
- net SD_D2: now reaches U1.78 (PC10)
- net SD_D2: now also Card1.1 (DAT2), D6.1 (IO1), R22.1
- net SD_D3: now reaches U1.79 (PC11)
- net SD_D3: now also Card1.2 (CD/DAT3), D6.2 (IO2), R23.1
- net SD_CLK: now reaches U1.80 (PC12)
- net SD_CLK: now also Card1.5 (CLK), D6.5 (IO4)
- net CANRX1: now reaches U1.81 (PD0)
- net CANTX1: now reaches U1.82 (PD1)
- net SD_CMD: now reaches U1.83 (PD2)
- net SD_CMD: now also U1.87 (PD6), Card1.3 (CMD), D6.3 (IO3), R24.1
- net CANRX2: now reaches U1.91 (PB5)
- net CANTX2: now reaches U1.92 (PB6)
- net GPIO_DOUT0: now reaches U1.97 (PE0)
- net GPIO_DOUT0: now also R13.1
- net GPIO_DOUT1: now reaches U1.98 (PE1)
- net GPIO_DOUT1: now also R16.1
- net +5V renamed 4.5V
- net 4.5V: now also C21.1, C24.1, C50.2, C51.2
- net 12VGPIO renamed 12VGPIO0
- net Brake1 renamed 5VAIN1
- net 5VAIN1: now also R65.1
- net Brake2 renamed 5VAIN0
- net 5VAIN0: now also R62.1
- net PA10 (ID): no longer names the net of U23.4 (I/O3)
- net PA10 (ID): no longer J7.4 (ID)
- net Temp1 renamed 5VAIN7
- net 5VAIN7: now also R68.1
- net Throttle1 renamed 5VAIN4
- net 5VAIN4: now also R84.1
- net Throttle2 renamed 5VAIN2
- net 5VAIN2: now also R72.1
- net fan_PWM_12V renamed DOUT1
- net DOUT1: now also Q3.3 (D)
- net pump_PWM_12V renamed DOUT0
- net DOUT0: now also Q2.3 (D)
- new net: Q3.1 (G), R16.2, R18.2
- new net: R37.1, U11.4
- new net: D9.3, R62.2, R63.1, R64.2
- new net: R55.1, U18.4
- new net: R33.2, U10.1
- new net: R46.2, U15.1
- new net: R51.2, U17.1
- new net: R52.1, U17.4
- new net: D8.3, R17.2, R60.2, R61.1
- new net: R20.1, S1.1 (A)
- new net: R31.1, U9.4
- new net: Q6.1 (G), R100.2, R101.2
- new net: Q2.1 (G), R13.2, R15.2
- new net: D18.3, R90.2, R91.1, R92.2
- new net: R58.1, U19.4
- new net: R40.1, U12.4
- new net: D10.3, R65.2, R66.1, R67.2
- new net: R47.1, U15.4
- new net: Q8.1 (G), R106.2, R107.2
- new net: D17.3, R87.2, R88.1, R89.2
- new net: R54.2, U18.1
- new net: R57.2, U19.1
- new net: D12.3, R72.2, R73.1, R74.2
- new net: Q5.1 (G), R97.2, R98.2
- new net: D13.3, R75.2, R76.1, R77.2
- new net: LED1.2 (K), R28.2
- new net: R34.1, U10.4
- new net: Q9.1 (G), R109.2, R110.2
- new net: R42.2, U13.1
- new net: R43.1, U13.4
- new net: D16.3, R84.2, R85.1, R86.2
- new net: Q7.1 (G), R103.2, R104.2
- new net: D15.3, R81.2, R82.1, R83.2
- new net: D1.2 (A), Q1.1 (G), R21.1
- new net: R36.2, U11.1
- new net: D11.3, R68.2, R69.1, R70.2
- new net: Q4.1 (G), R19.2, R96.2
- new net: R44.2, U14.1
- new net: D14.3, R78.2, R79.1, R80.2
- new net: R39.2, U12.1
- new net: D19.3, R93.2, R94.1, R95.2
- new net: R45.1, U14.4
- new net: R48.2, U16.1
- new net: R30.2, U9.1
- new net: R49.1, U16.4
- new net: Q1.2 (D), U7.2
- new net 12VGPIO1: R31.2, R32.1
- new net 12VGPIO2: R34.2, R35.1
- new net 12VGPIO3: R37.2, R38.1
- new net 12VGPIO4: R40.2, R41.1
- new net 12VGPIO5: R111.1, R43.2
- new net 12VGPIO6: R112.1, R45.2
- new net 12VGPIO7: R113.1, R47.2
- new net 5VAIN10: R87.1
- new net 5VAIN11: R93.1
- new net 5VAIN6: R60.1
- new net 5VAIN8: R75.1
- new net 5VAIN9: R81.1
- no-connect marks 5 -> 4
Other:
- note added: "100mA"
- note added: "12-4.5V 2A buck converter"
- note added: "12V DIN 0-7"
- note added: "12V High Side DOUT 4-5 Slow Rise"
- note added: "12V High Side DOUT 6-7 Fast Rise"
- note added: "12V Low Side DOUT 0-3"
- note added: "2A"
- note added: "3. Converts to 4.5V"
- note added: "4.5V-3.3V, 1.2A, MaxVin 18V"
- note added: "5V AIN 0-11"
- note added: "5V DIN 8-11"
- note added: "BMSfault"
- note added: "Brake1"
- note added: "Brake2"
- note added: "Copy BMS power architecture No bulk capcitance"
- note added: "Does fan control match current harness"
- note added: "ESD"
- note added: "IMDfault"
- note added: "Keep the Vout pour large for thermals"
- note added: "Micro-SD CARD - card detevt on pa7"
- note added: "NRST is normally pulled up. If NRST==0, then rest board. This triggered by button or ESP32 OTA PROG"
- note added: "Need footprint"
- note added: "No 5V on this board. 4.5V for lower heat"
- note added: "No CAN FD"
- note added: "PWM POWER OUTPUT"
- note added: "TSMS"
- note added: "Temp1"
- note added: "Temp2"
- note added: "Throttle1"
- note added: "Throttle2"
- note added: "Voltage divider sets Vout = 4.48V"
- note removed: "12-5V 2A buck converter"
- note removed: "12V Buck ~ 1.6A 4 12V Outputs ~ 4 x 100mA 2A, upsize to 5A for temp headroom"
- note removed: "3. Converts to 5V"
- note removed: "5V-3.3V, 1.2A, MaxVin 18V"
- note removed: "Analog Inputs"
- note removed: "Digital Inputs"
- note removed: "Do i need to breakout NRST for OTA?"
- note removed: "I oversized capacitor to account for any capacitance loss due to ceramic"
- note removed: "Low active SPI"
- note removed: "Micro-SD CARD"
- note removed: "Need to add BOOT0 control to esp32. then update pull up resistor to avoid voltage divider"
- note removed: "Reference document"
- note removed: "pull up resistors for data lines (47k)"
- moved on the sheet: C15, C25, C26, C27, C28, C29, C31, D2, D3, J7, L4, L5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
