File: 2026-27/Boards/VIL_RML/VIL_RML.kicad_sch (KiCad schematic)
At the start: 9 parts, among them Q5 UJ3N065080K3S

Commit message: Add hierarchical sheets to VIL RML
Parts:
- removed D10: H11L1M_LED, symbol Device:LED
- removed D2: 1N4148WT, Diode_SMD:D_SOD-523, symbol Diode:1N4148WT
- removed D6: PESD12VL1BA, Diode_SMD:D_SOD-323, symbol Diode:1.5KExxCA
- removed D8: BZT52C51, Diode_SMD:D_SOD-123F, symbol Diode:BZT52Bxx
- removed D9: LED, symbol Device:LED
- removed Q5: UJ3N065080K3S, Package_TO_SOT_THT:TO-247-3_Horizontal_TabDown, symbol Simulation_SPICE:NJFET
- removed R2: 2k, Resistor_SMD:R_0805_2012Metric_Pad1.20x1.40mm_HandSolder, symbol Device:R
- removed R3: 5600, Resistor_SMD:R_0805_2012Metric_Pad1.20x1.40mm_HandSolder, symbol Device:R
- removed V1: 400, symbol Simulation_SPICE:VDC
- added C1: 0.1uF, Capacitor_SMD:C_0805_2012Metric_Pad1.18x1.45mm_HandSolder, symbol Device:C
- added C3: 1uF, Capacitor_SMD:C_0805_2012Metric_Pad1.18x1.45mm_HandSolder, symbol Device:C
- added C4: 100uF, Capacitor_SMD:CP_Elec_6.3x5.4, symbol Device:C_Polarized
- added D1: 1N4148WT, Diode_SMD:D_SOD-523, symbol Diode:1N4148WT
- added D3: BZT52C51, Diode_SMD:D_SOD-123F, symbol Diode:BZT52Bxx
- added D4: PESD12VL1BA, Diode_SMD:D_SOD-323, symbol Diode:1.5KExxCA
- added F1, F2: 750mA, Fuse:Fuse_1206_3216Metric, symbol Device:Fuse
- added H1, H2, H3, H4: MountingHole, MountingHole:MountingHole_3.2mm_M3, symbol Mechanical:MountingHole
- added J1: 043045-0412, Connector_Molex:Molex_Micro-Fit_3.0_43045-0412_2x02_P3.00mm_Vertical, symbol Connector_Generic:Conn_01x04
- added LED1, Molex1: 043045-0212, Connector_Molex:Molex_Micro-Fit_3.0_43045-0212_2x01_P3.00mm_Vertical, symbol Connector_Generic:Conn_01x02
- added Q2, Q4: AO3401A, Package_TO_SOT_SMD:SOT-23, symbol Transistor_FET:AO3400A
- added Q3: UJ3N065080K3S, Package_TO_SOT_THT:TO-247-3_Horizontal_TabDown, symbol Simulation_SPICE:NJFET
- added R1, R9: 2k, Resistor_SMD:R_0805_2012Metric_Pad1.20x1.40mm_HandSolder, symbol Device:R
- added R4, R8: 1k, Resistor_SMD:R_0805_2012Metric_Pad1.20x1.40mm_HandSolder, symbol Device:R
- added R5: 100, Resistor_SMD:R_0805_2012Metric_Pad1.20x1.40mm_HandSolder, symbol Device:R
- added R6: 5.6k, Resistor_SMD:R_0805_2012Metric_Pad1.20x1.40mm_HandSolder, symbol Device:R
- added R7: 3k, Resistor_SMD:R_0805_2012Metric_Pad1.20x1.40mm_HandSolder, symbol Device:R
- added U1: H11L1M, Package_DIP:DIP-6_W7.62mm, symbol Isolator:H11L1
- added U2: NE555D, Package_SO:SOIC-8_3.9x4.9mm_P1.27mm, symbol Timer:NE555D
Connections:
- net GND: now also C1.1, C3.1, C4.2, J1.2 (Pin_2), R8.1, U1.5, U2.1 (GND)
- new net: D3.1 (K), F1.2
- new net: D3.2 (A), Q3.2 (D)
- new net: C4.1, R7.1, U2.2 (TR), U2.6 (THR)
- new net: Q2.1 (G), R4.1, U2.3 (Q)
- new net: Q4.3 (D), R5.1, R8.2, U2.4 (R)
- new net: C1.2, U2.5 (CV)
- new net: R5.2, R7.2, U2.7 (DIS)
- new net: Q4.1 (G), R1.2, U1.4
- new net: D1.1 (K), D4.1 (A1), Q3.3 (S), R6.1, R9.1
- new net: R6.2, U1.1
- new net: LED1.1 (Pin_1), R9.2
- new net: F2.2, Molex1.1 (Pin_1)
- new net GLV+: C3.2, J1.1 (Pin_1), Q2.3 (D), Q4.2 (S), R1.1, R4.2, U1.6, U2.8 (VCC)
- new net HV+: F1.1, Molex1.2 (Pin_2)
- new net HV-: D1.2 (A), D4.2 (A2), F2.1, LED1.2 (Pin_2), Q3.1 (G), U1.2
- new net Light+: J1.3 (Pin_3), Q2.2 (S)
- no-connect marks 0 -> 1
Other:
- added sheet HV Simulation (HV-sim.kicad_sch)
- added sheet LV-timer Simulation (LV-Sim.kicad_sch)
- note added: "HV+"
- note added: "HV-"
- note added: "NE555 Timer at ~3.3 Hz"
- note removed: ".model H11L1M_LED D(Is=1e-12 N=2 Rs=1 Eg=1.42 Cjo=100p Bv=6 Ibv=10u)"
- note removed: ".model led D(Is=1e-18 N=2 Rs=2 Eg=1.8 Cjo=10p Bv=5 Ibv=10u)"
- note removed: "HV_fused"
- note removed: "Simulation"
