File: 2026-27/Boards/BMS_Daughterboard_2027/BMS_Daughterboard_2027.kicad_sch (KiCad schematic)
At the start: 144 parts, among them CN2 0530470210, CN3 0530470210, Q1 ZXTN4004KTC, U1 BQ79616PAPRQ1

Commit message: daughterboard work
Parts:
- removed R33: RTT12100JTP, easyeda2kicad:R1210, symbol easyeda2kicad:RTT12100JTP
- removed R43, R44: 680Ω, PCM_JLCPCB:R_0402, symbol PCM_JLCPCB-Resistors:0402,680Ω
- removed TP1, TP25, TP26, TP27, TP28, TP29: TestPoint_Small, TestPoint:TestPoint_Pad_D1.0mm, symbol Connector:TestPoint_Small
- added CN1, CN4, CN5, CN6, CN7, CN8: BM02B-SRSS-TB, FSAE:CONN-TH_BM02B-SRSS-TB-LF-SN, symbol FSAE:BM02B-SRSS-TB
- added D10, D5, D6, D7, D8, D9: NTC_Diode, symbol Device:D_TemperatureDependent_Filled
- added Q2, Q3, Q4: DMN2005DLP4K-7, FSAE:X2-DFN1310-6_L1.3-W1.0-P0.35-BL, symbol FSAE:DMN2005DLP4K-7
- added R21: RTT12100JTP, FSAE:C1206, symbol easyeda2kicad:RTT12100JTP
- added R47, R48, R49, R50: 680Ω, PCM_JLCPCB:R_0402, symbol PCM_JLCPCB-Resistors:0402,680Ω
- D1, D2: footprint easyeda2kicad:SMD-6_L7.6-W6.9-P2.54-LS8.9-BL -> FSAE:SMD-6_L7.6-W6.9-P2.54-LS8.9-BL
- L2: footprint easyeda2kicad:FILTER-SMD_4P-L4.5-W3.2-TL_ACT45B -> FSAE:FILTER-SMD_4P-L4.5-W3.2-TL_ACT45B
- Q1: footprint easyeda2kicad:TO-252-2_L6.6-W6.1-P4.58-LS9.9-TL -> PCM_JLCPCB:TO-252-2_L6.5-W6.1-P4.58-LS10.0-TL
- R20, R22, R23, R24, R25, R26, R27, R28, R29, R30, R31, R32: footprint easyeda2kicad:R1210 -> FSAE:C1206
Connections:
- net CB0: now also R32.2; no longer R29.2
- net CB1: now also R31.2
- net CB11: now also R21.2; no longer R24.2
- net CB2: now also R30.2; no longer R28.2
- net CB3: now also R29.2; no longer R32.2
- net CB4: now also R28.2; no longer R27.2
- net CB5: now also R27.2; no longer R31.2
- net CB7: now also R25.2; no longer R30.2
- net CB8: now also R24.2; no longer R23.2
- net CB9: now also R23.2; no longer R25.2
- net CELL1+: now also R31.1
- net CELL1-: now also R32.1; no longer R29.1
- net CELL11+: now also R21.1; no longer R24.1
- net CELL2+: now also R30.1; no longer R28.1
- net CELL3+: now also R29.1; no longer R32.1
- net CELL4+: now also R28.1; no longer R27.1
- net CELL5+: now also R27.1; no longer R31.1
- net CELL7+: now also R25.1; no longer R30.1
- net CELL8+: now also R24.1; no longer R23.1
- net CELL9+: now also R23.1; no longer R25.1
- net GND: now also Q2.1 (S1), Q2.4 (S2), Q3.1 (S1), Q3.4 (S2), Q4.1 (S1), Q4.4 (S2)
- net TSREF: now also Q2.2 (G1), Q2.5 (G2), Q3.2 (G1), Q3.5 (G2), Q4.2 (G1), Q4.5 (G2); no longer R41.2, R42.2
- net temp6+: now reaches U1.56 (GPIO6)
- net temp6+: now also CN8.2, R50.1
- net temp5+: now reaches U1.57 (GPIO5)
- net temp5+: now also CN7.2, R49.1
- net temp1 renamed temp1+
- net temp1+: now also CN1.2
- net temp2 renamed temp2+
- net temp2+: now also CN4.2
- net temp3 renamed temp3+
- net temp3+: now also CN5.2, R47.1
- net temp4 renamed temp4+
- net temp4+: now also CN6.2, R48.1
- new net 3.3V: R41.2, R42.2, R47.2, R48.2, R49.2, R50.2
- new net temp1-: CN1.1, Q2.6 (D1)
- new net temp2-: CN4.1, Q2.3 (D2)
- new net temp3-: CN5.1, Q3.6 (D1), Q4.6 (D1)
- new net temp4-: CN6.1, Q3.3 (D2), Q4.3 (D2)
- new net temp5-: CN7.1
- new net temp6-: CN8.1
- no-connect marks 7 -> 19
Other:
- note added: "TEMP SENSORS"

Commit message: erc fixes for daughterboard pcba
Parts:
- removed C24, C80, C81, C82: 470nF, PCM_JLCPCB:C_0603, symbol PCM_JLCPCB-Capacitors:0603,470nF
- added C29: 470nF, PCM_JLCPCB:C_0603, symbol PCM_JLCPCB-Capacitors:0603,470nF
- added R3, R4: 10k, symbol Device:R
- added R33: RTT12100JTP, FSAE:C1206, symbol easyeda2kicad:RTT12100JTP
- H10, H11, H12, H14, H15, H16, H17, H18, H19, H21, H8: symbol Mechanical:MountingHole_Pad -> Mechanical:MountingHole
Connections:
- net CB13 is gone; now on net BAT: C79.1, U1.8 (CB13)
- net CB14 is gone; now on net BAT: U1.6 (CB14)
- net CB15 is gone; now on net BAT: U1.4 (CB15)
- net VC13 is gone; now on net BAT: U1.9 (VC13)
- net VC14 is gone; now on net BAT: U1.7 (VC14)
- net VC15 is gone; now on net BAT: U1.5 (VC15)
- net VC16 is gone; now on net BAT: U1.3 (VC16)
- net BAT: now also C29.2, R33.1
- net CB16: now also C29.1, R33.2
- net GND: now also R3.2, R4.2
- net temp3-: no longer Q4.6 (D1)
- net temp4-: no longer Q4.3 (D2)
- net temp5-: now also Q4.6 (D1)
- net temp6-: now also Q4.3 (D2)
- net at U1.54 (GPIO8): now also R4.1
- net at U1.55 (GPIO7): now also R3.1
- no-connect marks 19 -> 31
Other:
- note added: "temporarily added no connect flags"
- moved on the sheet: C25, C28, C30, C32, C4, C7, C79, R80

Commit message: daughterboard cell tap connector
Parts:
- removed CN1, CN4, CN5, CN6, CN7, CN8: BM02B-SRSS-TB, FSAE:CONN-TH_BM02B-SRSS-TB-LF-SN, symbol FSAE:BM02B-SRSS-TB
- removed D10, D5, D6, D7, D8, D9: NTC_Diode, symbol Device:D_TemperatureDependent_Filled
- removed F1, F10, F11, F12, F13, F2, F3, F4, F5, F6, F7, F8, F9: JFC2410-1125FS, FSAE:FUSE-SMD_JFC2410-1150FS_C2994707, symbol FSAE:JFC2410-1125FS
- removed H1, H13, H2, H20, H22, H23, H24, H3, H4, H5, H6, H7, H9: MountingHole_Pad, MountingHole:MountingHole_5.5mm_M5_Pad_Via, symbol Mechanical:MountingHole_Pad
- removed H10, H11, H12, H14, H15, H16, H17, H18, H19, H21, H8: MountingHole_Pad, MountingHole:MountingHole_5.5mm_M5_Pad_Via, symbol Mechanical:MountingHole
- removed Q2, Q3, Q4: DMN2005DLP4K-7, FSAE:X2-DFN1310-6_L1.3-W1.0-P0.35-BL, symbol FSAE:DMN2005DLP4K-7
- removed R41, R42, R47, R48, R49, R50: 680Ω, PCM_JLCPCB:R_0402, symbol PCM_JLCPCB-Resistors:0402,680Ω
- added J1: 5031543090, CONN_503154_30_MOL, symbol FSAE:5031543090
Connections:
- net CELL1+: now also J1.15
- net CELL1-: now also J1.11
- net CELL10+: now also J1.17
- net CELL11+: now also J1.23
- net CELL12+: now also J1.25; no longer R1.2, R77.2, R80.2
- net CELL2+: now also J1.19
- net CELL3+: now also J1.29
- net CELL4+: now also J1.3
- net CELL5+: now also J1.21
- net CELL6+: now also J1.1
- net CELL7+: now also J1.5
- net CELL8+: now also J1.7
- net CELL9+: now also J1.9
- net GND: now also J1.13
- net temp1+: now also J1.2
- net temp1-: now also J1.4
- net temp2+: now also J1.28
- net temp2-: now also J1.30
- net temp3+: now also J1.6
- net temp3-: now also J1.8
- net temp4+: now also J1.24
- net temp4-: now also J1.26
- net temp5+: now also J1.10
- net temp5-: now also J1.12
- net temp6+: now also J1.20
- net temp6-: now also J1.22
- new net CELL_TOP: J1.27, R1.2, R77.2, R80.2
- no-connect marks 31 -> 10
Other:
- note added: "TO CELL TAP BOARD"
- note removed: "FUSES"
- note removed: "TEMP SENSORS"
- note removed: "temporarily added no connect flags"

Commit message: 2027 Daughterboard for review
Parts:
- removed R3, R4: 10k, symbol Device:R
- added R24, R25, R26, R27, R28, R29, R30, R31: RC0603FR-0710KL, FSAE:R0603, symbol FSAE:RC0603FR-0710KL
- renumbered C43 to C1, C47 to C10, C79 to C11, C32 to C12, C33 to C13, C38 to C14, C39 to C15, C40 to C16, C41 to C17, C29 to C18, C45 to C19, C44 to C2, C46 to C20, C77 to C21, C48 to C22, C49 to C23, C7 to C24, C6 to C25, C25 to C26, C78 to C27, C1 to C28, C5 to C29, C28 to C3, C4 to C30, C2 to C31, C50 to C32, C51 to C33, C52 to C34, C13 to C35, C16 to C36, C17 to C37, C18 to C38, C19 to C39, C30 to C4, C8 to C40, C14 to C41, C15 to C42, C20 to C43, C21 to C44, C22 to C45, C23 to C46, C72 to C47, C31 to C5, C34 to C6, C35 to C7, C36 to C8, C37 to C9, CN2 to CN1, CN3 to CN2, D3 to D1, D1 to D2, D4 to D3, D2 to D4, JP4 to JP1, JP3 to JP2, R35 to R1, R32 to R10, R21 to R11, R23 to R12, R25 to R13, R27 to R14, R29 to R15, R31 to R16, R33 to R17, R1 to R18, R77 to R19, R36 to R2, R38 to R20, R80 to R21, R39 to R22, R40 to R23, R37 to R3, R6 to R32, R7 to R33, R8 to R34, R9 to R35, R10 to R36, R11 to R37, R12 to R38, R13 to R39, R20 to R4, R14 to R40, R15 to R41, R16 to R42, R17 to R43, R2 to R44, R22 to R5, R24 to R6, R26 to R7, R28 to R8, R30 to R9
Connections:
- net temp1- is gone; now on net GND: J1.4
- net temp2- is gone; now on net GND: J1.30
- net temp3- is gone; now on net GND: J1.8
- net temp4- is gone; now on net GND: J1.26
- net temp5- is gone; now on net GND: J1.12
- net temp6- is gone; now on net GND: J1.22
- net GND: now also R24.2, R25.2
- net TSREF: now also R26.2, R27.2, R28.2, R29.2, R30.2, R31.2
- net temp1+: now also R26.1
- net temp2+: now also R27.1
- net temp3+: now also R28.1
- net temp4+: now also R29.1
- net temp5+: now also R30.1
- net temp6+: now also R31.1
- net at JP2.1 (A): now also R19.1; no longer R18.1
- net at JP1.1 (A): now also R18.1; no longer R19.1
- net at U1.54 (GPIO8): now also R25.1
- net at U1.55 (GPIO7): now also R24.1
- no-connect marks 10 -> 9
Other:
- note added: "CELL TAP CONNECTOR"
- note added: "swapped JP3 & JP4 for 12cell, was devboard 6cell ?"
- note added: "temp return to gnd"
- note added: "temp sense to GPIOs (pulled up to TSREF)"
- note added: "this should be rated for full segment voltage ?"
- note removed: "TO CELL TAP BOARD"
- moved on the sheet: C10, C21, C24, C25, C26, C27, C28, C29, C30, C31, C32, JP1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

Commit message: fixed connector pn
Parts:
- J1: footprint CONN_503154_30_MOL -> FSAE:CONN-TH_5018763040; symbol FSAE:5031543090 -> FSAE:5018763040; LCSC Part (none) -> C293585; MPN (none) -> 5018763040; Manufacturer (none) -> MOLEX
Connections:
- net collector: no longer JP1.2 (B), JP2.2 (B)
- net at JP2.1 (A): no longer R19.1
- net at JP1.1 (A): no longer R18.1
- no-connect marks 9 -> 11
Other:
- note removed: "swapped JP3 & JP4 for 12cell, was devboard 6cell ?"
- note removed: "temp return to gnd"
- note removed: "temp sense to GPIOs (pulled up to TSREF)"
