File: 2026-27/Boards/Celltap_Boards/Negative_Celltap_2027/Negative_Celltap_2027.kicad_pcb (KiCad board)
At the start: 4 copper layers, 206.5 x 79 mm, 42 parts, among them J1 5031543090, U1 SMTSO40100CTJ, U2 SMTSO40100CTJ, U3 SMTSO40100CTJ, U4 SMTSO40100CTJ

Commit message: Negative Celltap board 2027 for review
Parts:
- added F0: JFC2410-1125FS, FSAE:FUSE-SMD_JFC2410-1150FS_C2994707, F.Cu at (146.8, 61.7)
- added F14: JFC2410-1125FS, FSAE:FUSE-SMD_JFC2410-1150FS_C2994707, F.Cu at (146.8, 21.1)
- added J2: 533984002, FSAE:CONN_533980002-SD_02_MOL, F.Cu at (50.7, 71.9)
- added J3: 533984002, FSAE:CONN_533980002-SD_02_MOL, F.Cu at (50.4, 30.8)
- added J4: 533984002, FSAE:CONN_533980002-SD_02_MOL, F.Cu at (104.8, 71.8)
- added J5: 533984002, FSAE:CONN_533980002-SD_02_MOL, F.Cu at (104.8, 31.2)
- added J6: 533984002, FSAE:CONN_533980002-SD_02_MOL, F.Cu at (173.8, 68.7)
- added J7: 533984002, FSAE:CONN_533980002-SD_02_MOL, F.Cu at (173.8, 34.4)
- H1, H10, H11, H12, H13, H14, H15, H16, H17, H18, H19, H2, H20, H21, H22, H23, H24, H3, H4, H5, H6, H7, H8, H9: footprint MountingHole:MountingHole_5.5mm_M5_Pad_Via -> MountingHole:MountingHole_5.5mm_Pad_Via
- moved U4 117.3 mm to (115.2, 81.4)
- moved U3 110.1 mm to (115.2, 21.5)
- moved F2 69.3 mm to (146.8, 41.4)
- moved F1 68.2 mm to (81.8, 61.7), turned to 90 degrees
- moved F6 66.4 mm to (20.3, 71.8), turned to 0 degrees
- moved U2 62.3 mm to (34.7, 71.9)
- moved F8 61.3 mm to (147.6, 82.5)
- moved F4 61.3 mm to (20.3, 31.2), turned to 180 degrees
- moved F12 60.3 mm to (153.3, 21.1)
- moved F9 56.6 mm to (198.0, 81.8)
- moved F5 51.2 mm to (79.3, 41.4)
- moved J1 49.4 mm to (45.8, 51.5), turned to -90 degrees
- moved F3 49.3 mm to (81.8, 21.1)
- moved U1 38.7 mm to (34.4, 30.8)
- moved F7 32.2 mm to (57.3, 82.0), turned to 90 degrees
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Connections:
- F1 pad 2: Net-(F1-Pad2) -> /F1
- F10 pad 2: Net-(F10-Pad2) -> /F10
- F11 pad 2: Net-(F11-Pad2) -> /F11
- F12 pad 2: Net-(F12-Pad2) -> /F12
- F13 pad 1: Net-(F13-Pad1) -> Net-(F0-Pad1)
- F13 pad 2: Net-(F13-Pad2) -> /F_GND
- F2 pad 2: Net-(F2-Pad2) -> /F2
- F3 pad 2: Net-(F3-Pad2) -> /F3
- F4 pad 2: Net-(F4-Pad2) -> /F4
- F5 pad 2: Net-(F5-Pad2) -> /F5
- F6 pad 1: Net-(F6-Pad1) -> /F6
- F7 pad 2: Net-(F7-Pad2) -> /F7
- F8 pad 2: Net-(F8-Pad2) -> /F8
- F9 pad 2: Net-(F9-Pad2) -> /F9
- H1 pad 1: Net-(F1-Pad1) -> Net-(F0-Pad1)
- H10 pad 1: Net-(F10-Pad2) -> Net-(F9-Pad1)
- H11 pad 1: Net-(F11-Pad2) -> Net-(F10-Pad1)
- H12 pad 1: Net-(F12-Pad2) -> Net-(F11-Pad1)
- H13 pad 1: Net-(F13-Pad2) -> Net-(F12-Pad1)
- H2 pad 1: Net-(F2-Pad1) -> Net-(F1-Pad1)
- H3 pad 1: Net-(F3-Pad1) -> Net-(F2-Pad1)
- H4 pad 1: Net-(F4-Pad1) -> Net-(F3-Pad1)
- H5 pad 1: Net-(F5-Pad1) -> Net-(F4-Pad1)
- H6 pad 1: Net-(F6-Pad1) -> Net-(F5-Pad1)
- H7 pad 1: Net-(F7-Pad2) -> Net-(F6-Pad2)
- H8 pad 1: Net-(F8-Pad2) -> Net-(F7-Pad1)
- H9 pad 1: Net-(F9-Pad2) -> Net-(F8-Pad1)
- J1 pad 1: Net-(F1-Pad2) -> /F6
- J1 pad 10: Net-(F10-Pad2) -> /Temp5_Sense
- J1 pad 11: Net-(F11-Pad2) -> /F0
- J1 pad 12: Net-(F12-Pad2) -> /Temp5_Return
- J1 pad 13: Net-(F13-Pad2) -> /F_GND
- J1 pad 15: unconnected-(J1-Pad15) -> /F1
- J1 pad 17: unconnected-(J1-Pad17) -> /F10
- J1 pad 19: unconnected-(J1-Pad19) -> /F2
- J1 pad 2: Net-(F2-Pad2) -> /Temp1_Sense
- J1 pad 20: unconnected-(J1-Pad20) -> /Temp6_Sense
- J1 pad 21: unconnected-(J1-Pad21) -> /F5
- J1 pad 22: unconnected-(J1-Pad22) -> /Temp6_Return
- J1 pad 23: unconnected-(J1-Pad23) -> /F11
- J1 pad 24: unconnected-(J1-Pad24) -> /Temp4_Sense
- J1 pad 25: unconnected-(J1-Pad25) -> /F12
- J1 pad 26: unconnected-(J1-Pad26) -> /Temp4_Return
- J1 pad 27: unconnected-(J1-Pad27) -> /F_CELLTOP
- J1 pad 28: unconnected-(J1-Pad28) -> /Temp2_Sense
- J1 pad 29: unconnected-(J1-Pad29) -> /F3
- J1 pad 3: Net-(F3-Pad2) -> /F4
- J1 pad 30: unconnected-(J1-Pad30) -> /Temp2_Return
- J1 pad 4: Net-(F4-Pad2) -> /Temp1_Return
- J1 pad 5: Net-(F5-Pad2) -> /F7
- J1 pad 6: Net-(F6-Pad2) -> /Temp3_Sense
- J1 pad 7: Net-(F7-Pad1) -> /F8
- J1 pad 8: Net-(F8-Pad2) -> /Temp3_Return
- J1 pad 9: Net-(F9-Pad2) -> /F9
Routing:
- net /F9: track 0.00 -> 173.5 mm, vias 0 -> 2
- net /F11: track 0.00 -> 171.8 mm, vias 0 -> 2
- net /Temp5_Return: track 0.00 -> 135.3 mm, vias 0 -> 2
- net /Temp6_Sense: track 0.00 -> 134.9 mm, vias 0 -> 2
- net /Temp5_Sense: track 0.00 -> 132.5 mm, vias 0 -> 2
- net /Temp6_Return: track 0.00 -> 132.1 mm, vias 0 -> 2
- net /F12: track 0.00 -> 128.4 mm, vias 0 -> 2
- net /F10: track 0.00 -> 123.2 mm, vias 0 -> 2
- net /F8: track 0.00 -> 122.5 mm, vias 0 -> 2
- net /F0: track 0.00 -> 122.5 mm, vias 0 -> 2
- net /F_CELLTOP: track 0.00 -> 121.2 mm, vias 0 -> 2
- net /F2: track 0.00 -> 116.6 mm, vias 0 -> 2
- net /F_GND: track 0.00 -> 80.2 mm, vias 0 -> 2
- net /Temp3_Return: track 0.00 -> 62.0 mm
- net /Temp3_Sense: track 0.00 -> 62.0 mm
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Other:
- outline, holes or cut-outs redrawn
- board text added: "Negative Celltap PCBA SCFE 27 Accumulator"
- board text removed: "{dblquote}Negative{dblquote} Celltap PCBA SCFE 27 Accumulator"

Commit message: celltap pcba positive first draft for review
Parts:
- moved U1 0.95 mm to (35.3, 31.2)
- moved U2 0.56 mm to (35.3, 71.8)
- moved U4 0.56 mm to (115.3, 82.0)
- moved U3 0.45 mm to (115.3, 21.1)
Other:
- board text added: "Negative Celltap PCBA SCFE 27 HVBP"
- board text removed: "Negative Celltap PCBA SCFE 27 Accumulator"
