File: 2026-27/Boards/Celltap_Boards/Positive_Celltap_2027/Positive_Celltap_2027.kicad_sch (KiCad schematic)
At the start: 38 parts, among them J1 5016451420

Commit message: positive cell taps
Parts:
- removed F10, F11, F12, F13, F8, F9: 885001, 885001_Littelfusefootprints:FUSC10948X488N, symbol 885001:885001
- added F10, F11, F12, F13, F14, F7, F8, F9: JFC2410-1125FS, FSAE:FUSE-SMD_JFC2410-1150FS_C2994707, symbol FSAE:JFC2410-1125FS
- added J2, J3, J4, J5, J6, J7: 533984002, FSAE:CONN_533980002-SD_02_MOL, symbol FSAE:533984002
- added U1, U2, U3, U4: SMTSO40100CTJ, FSAE:SMD_SMTSO40100CTJ, symbol FSAE:SMTSO40100CTJ
- F0: renamed from F1; value 885001 -> JFC2410-1125FS; footprint 885001_Littelfusefootprints:FUSC10948X488N -> FSAE:FUSE-SMD_JFC2410-1150FS_C2994707; symbol 885001:885001 -> FSAE:JFC2410-1125FS; Height 4.88 -> (none); LCSC Part (none) -> C55058772; MPN (none) -> JFC2410-1125FS; Manufacturer (none) -> JDTfuse(集电通); Manufacturer_Name LITTELFUSE -> (none); Manufacturer_Part_Number 885001 -> (none)
- F1: renamed from F2; value 885001 -> JFC2410-1125FS; footprint 885001_Littelfusefootprints:FUSC10948X488N -> FSAE:FUSE-SMD_JFC2410-1150FS_C2994707; symbol 885001:885001 -> FSAE:JFC2410-1125FS; Height 4.88 -> (none); LCSC Part (none) -> C55058772; MPN (none) -> JFC2410-1125FS; Manufacturer (none) -> JDTfuse(集电通); Manufacturer_Name LITTELFUSE -> (none); Manufacturer_Part_Number 885001 -> (none)
- F2: renamed from F3; value 885001 -> JFC2410-1125FS; footprint 885001_Littelfusefootprints:FUSC10948X488N -> FSAE:FUSE-SMD_JFC2410-1150FS_C2994707; symbol 885001:885001 -> FSAE:JFC2410-1125FS; Height 4.88 -> (none); LCSC Part (none) -> C55058772; MPN (none) -> JFC2410-1125FS; Manufacturer (none) -> JDTfuse(集电通); Manufacturer_Name LITTELFUSE -> (none); Manufacturer_Part_Number 885001 -> (none)
- F3: renamed from F4; value 885001 -> JFC2410-1125FS; footprint 885001_Littelfusefootprints:FUSC10948X488N -> FSAE:FUSE-SMD_JFC2410-1150FS_C2994707; symbol 885001:885001 -> FSAE:JFC2410-1125FS; Height 4.88 -> (none); LCSC Part (none) -> C55058772; MPN (none) -> JFC2410-1125FS; Manufacturer (none) -> JDTfuse(集电通); Manufacturer_Name LITTELFUSE -> (none); Manufacturer_Part_Number 885001 -> (none)
- F4: renamed from F5; value 885001 -> JFC2410-1125FS; footprint 885001_Littelfusefootprints:FUSC10948X488N -> FSAE:FUSE-SMD_JFC2410-1150FS_C2994707; symbol 885001:885001 -> FSAE:JFC2410-1125FS; Height 4.88 -> (none); LCSC Part (none) -> C55058772; MPN (none) -> JFC2410-1125FS; Manufacturer (none) -> JDTfuse(集电通); Manufacturer_Name LITTELFUSE -> (none); Manufacturer_Part_Number 885001 -> (none)
- F5: renamed from F6; value 885001 -> JFC2410-1125FS; footprint 885001_Littelfusefootprints:FUSC10948X488N -> FSAE:FUSE-SMD_JFC2410-1150FS_C2994707; symbol 885001:885001 -> FSAE:JFC2410-1125FS; Height 4.88 -> (none); LCSC Part (none) -> C55058772; MPN (none) -> JFC2410-1125FS; Manufacturer (none) -> JDTfuse(集电通); Manufacturer_Name LITTELFUSE -> (none); Manufacturer_Part_Number 885001 -> (none)
- F6: renamed from F7; value 885001 -> JFC2410-1125FS; footprint 885001_Littelfusefootprints:FUSC10948X488N -> FSAE:FUSE-SMD_JFC2410-1150FS_C2994707; symbol 885001:885001 -> FSAE:JFC2410-1125FS; Height 4.88 -> (none); LCSC Part (none) -> C55058772; MPN (none) -> JFC2410-1125FS; Manufacturer (none) -> JDTfuse(集电通); Manufacturer_Name LITTELFUSE -> (none); Manufacturer_Part_Number 885001 -> (none)
- H1: value MountingHole_Pad -> C1-; footprint MountingHole:MountingHole_5.5mm_M5_Pad_Via -> MountingHole:MountingHole_5.5mm_Pad_Via
- H10: value MountingHole_Pad -> C9+; footprint MountingHole:MountingHole_5.5mm_M5_Pad_Via -> MountingHole:MountingHole_5.5mm_Pad_Via
- H11: value MountingHole_Pad -> C10+; footprint MountingHole:MountingHole_5.5mm_M5_Pad_Via -> MountingHole:MountingHole_5.5mm_Pad_Via
- H12: value MountingHole_Pad -> C11+; footprint MountingHole:MountingHole_5.5mm_M5_Pad_Via -> MountingHole:MountingHole_5.5mm_Pad_Via
- H13: value MountingHole_Pad -> C12+; footprint MountingHole:MountingHole_5.5mm_M5_Pad_Via -> MountingHole:MountingHole_5.5mm_Pad_Via
- H14: value MountingHole_Pad -> C2-; footprint MountingHole:MountingHole_5.5mm_M5_Pad_Via -> MountingHole:MountingHole_5.5mm_Pad_Via
- H15: value MountingHole_Pad -> C3-; footprint MountingHole:MountingHole_5.5mm_M5_Pad_Via -> MountingHole:MountingHole_5.5mm_Pad_Via
- H16: value MountingHole_Pad -> C4-; footprint MountingHole:MountingHole_5.5mm_M5_Pad_Via -> MountingHole:MountingHole_5.5mm_Pad_Via
- H17: value MountingHole_Pad -> C5-; footprint MountingHole:MountingHole_5.5mm_M5_Pad_Via -> MountingHole:MountingHole_5.5mm_Pad_Via
- H18: value MountingHole_Pad -> C6-; footprint MountingHole:MountingHole_5.5mm_M5_Pad_Via -> MountingHole:MountingHole_5.5mm_Pad_Via
- H19: value MountingHole_Pad -> C7-; footprint MountingHole:MountingHole_5.5mm_M5_Pad_Via -> MountingHole:MountingHole_5.5mm_Pad_Via
- H2: value MountingHole_Pad -> C1+; footprint MountingHole:MountingHole_5.5mm_M5_Pad_Via -> MountingHole:MountingHole_5.5mm_Pad_Via
- H20: value MountingHole_Pad -> C8-; footprint MountingHole:MountingHole_5.5mm_M5_Pad_Via -> MountingHole:MountingHole_5.5mm_Pad_Via
- H21: value MountingHole_Pad -> C9-; footprint MountingHole:MountingHole_5.5mm_M5_Pad_Via -> MountingHole:MountingHole_5.5mm_Pad_Via
- H22: value MountingHole_Pad -> C10-; footprint MountingHole:MountingHole_5.5mm_M5_Pad_Via -> MountingHole:MountingHole_5.5mm_Pad_Via
- H23: value MountingHole_Pad -> C11-; footprint MountingHole:MountingHole_5.5mm_M5_Pad_Via -> MountingHole:MountingHole_5.5mm_Pad_Via
- H24: value MountingHole_Pad -> C12-; footprint MountingHole:MountingHole_5.5mm_M5_Pad_Via -> MountingHole:MountingHole_5.5mm_Pad_Via
- H3: value MountingHole_Pad -> C2+; footprint MountingHole:MountingHole_5.5mm_M5_Pad_Via -> MountingHole:MountingHole_5.5mm_Pad_Via
- H4: value MountingHole_Pad -> C3+; footprint MountingHole:MountingHole_5.5mm_M5_Pad_Via -> MountingHole:MountingHole_5.5mm_Pad_Via
- H5: value MountingHole_Pad -> C4+; footprint MountingHole:MountingHole_5.5mm_M5_Pad_Via -> MountingHole:MountingHole_5.5mm_Pad_Via
- H6: value MountingHole_Pad -> C5+; footprint MountingHole:MountingHole_5.5mm_M5_Pad_Via -> MountingHole:MountingHole_5.5mm_Pad_Via
- H7: value MountingHole_Pad -> C6+; footprint MountingHole:MountingHole_5.5mm_M5_Pad_Via -> MountingHole:MountingHole_5.5mm_Pad_Via
- H8: value MountingHole_Pad -> C7+; footprint MountingHole:MountingHole_5.5mm_M5_Pad_Via -> MountingHole:MountingHole_5.5mm_Pad_Via
- H9: value MountingHole_Pad -> C8+; footprint MountingHole:MountingHole_5.5mm_M5_Pad_Via -> MountingHole:MountingHole_5.5mm_Pad_Via
- J1: value 5016451420 -> 5031543090; footprint footprints:CONN14_5016451420_MOL -> FSAE:CONN_503154_30_MOL; symbol Molex_14pin_Female:5016451420 -> FSAE:5031543090
Connections:
- net at H13.1: now also F12.1, F14.1
- net at J1.3: no longer F2.2
- net at F0.1, H1.1: now also F13.1
- net at F6.1: now also H7.1; no longer J1.7
- net F6: now reaches F6.2
- net F6: no longer H7.1
- net at J1.1: no longer F0.2
- net at J1.2: no longer F1.2
- net at J1.4: no longer F3.2
- net at J1.5: no longer F4.2
- net at J1.6: no longer F5.2
- net at H9.1: now also F8.1
- net at H8.1: now also F7.1
- net at H10.1: now also F9.1
- net at H12.1: now also F11.1
- net at H11.1: now also F10.1
- new net F0: F0.2
- new net F1: F1.2
- new net F10: F10.2
- new net F11: F11.2
- new net F12: F12.2
- new net F2: F2.2
- new net F3: F3.2
- new net F4: F4.2
- new net F5: F5.2
- new net F7: F7.2
- new net F8: F8.2
- new net F9: F9.2
- new net F_CELLTOP: F14.2
- new net F_GND: F13.2
- new net Temp1_Return: J2.2
- new net Temp1_Sense: J2.1
- new net Temp2_Return: J3.2
- new net Temp2_Sense: J3.1
- new net Temp3_Return: J4.2
- new net Temp3_Sense: J4.1
- new net Temp4_Return: J5.2
- new net Temp4_Sense: J5.1
- new net Temp5_Return: J6.2
- new net Temp5_Sense: J6.1
- new net Temp6_Return: J7.2
- new net Temp6_Sense: J7.1
- no-connect marks 1 -> 4
Other:
- note added: "Standoffs M4x10"
- moved on the sheet: H1, H14, H15, H16, H17, H18, H19, H2, H3, H4, H5, H6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

Commit message: celltap pcba positive first draft for review
Connections:
- net F0: now also J1.11
- net F1: now also J1.15
- net F10: now also J1.17
- net F11: now also J1.23
- net F12: now also J1.25
- net F2: now also J1.19
- net F3: now also J1.29
- net F4: now also J1.3
- net F5: now also J1.21
- net F6: now also J1.1
- net F7: now also J1.5
- net F8: now also J1.7
- net F9: now also J1.9
- net F_CELLTOP: now also J1.27
- net F_GND: now also J1.13
- net Temp1_Return: now also J1.4
- net Temp1_Sense: now also J1.2
- net Temp2_Return: now also J1.30
- net Temp2_Sense: now also J1.28
- net Temp3_Return: now also J1.8
- net Temp3_Sense: now also J1.6
- net Temp4_Return: now also J1.26
- net Temp4_Sense: now also J1.24
- net Temp5_Return: now also J1.12
- net Temp5_Sense: now also J1.10
- net Temp6_Return: now also J1.22
- net Temp6_Sense: now also J1.20
- no-connect marks 4 -> 7
Other:
- moved on the sheet: F0, F1, F10, F11, F12, F13, F14, F2, F3, F4, F5, F6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
