File: 2026-27/Boards/VIL_RML/vil_rml_fullSIM/vil_rml_fullSIM.kicad_sch (KiCad schematic)
At the start: 21 parts, among them Q2 AO3401A, Q4 AO3401A, Q5 UJ3N065080K3S, U1 H11L1M, U2 NE555D

Commit message: rml/vil edit during workshop
Parts:
- added D10: LED, symbol Device:LED
- added R6: 2000, Resistor_SMD:R_0805_2012Metric_Pad1.20x1.40mm_HandSolder, symbol Device:R
- V2: value 5 -> 12
Connections:
- net Light+ is gone; now on net GND: Q2.2 (S)
- net GLV+: now also R6.1; no longer Q2.3 (D)
- new net: D10.1 (K), Q2.3 (D)
- new net: D10.2 (A), R6.2
