File: 2026-27/Schematics/Chargecart/Charge Cart + HVBP/chargecart_hvbp.kicad_sch (KiCad schematic)
At the start: 48 parts, among them J1 UPCR012ALS1, J11 UPCR012ALS1, J13 DTM04-12PA-L012, J2 DTM04-12PA-L012, J20 ??? can't find PN, J3 NEMA_5-20, J4 TSMP, J5 J1772, J7 DTM04-12PA-L012, K1 Charger Safety Relay, K2 GV24 1BAX, K3 P115 BDA, K4 GV24 1BAX, SW1 LV Switch, SW2 Charging Stop, SW4 Reset, U1 Milwaukee M12 Adapter, U12 IMD, U16 Battery Pack, U18 BMS, U19 DS18B20-PAR, U20 RSB, U3 Relay_Board, U4 6.6kW Elcon Charger, U5 Volt_indic, U6 Precharge

Commit message: fixed critical ERC
Connections:
- net GND is gone; now on net GLV-: R8.2
- net GNDPWR is gone; now on net GLV-: J13.3 (Pin_3), J2.4 (Pin_4), J2.5 (Pin_5), J3.3 (Ground), J5.3 (Ground), K2.2, MES1.1 (-), R3.1, SW1.2 (B), SW4.2, U12.1 (GND), U12.3 (GND), U12.4 (GND), U18. (GND_Lug), U18.11 (GND), U18.12 (GND), U3.2 (GND), U4.AC2 (Ground), U6.2 (GND), U6.4 (charge_on)
- net SDC1 is gone; now on net SDC4: J11.2 (Pin_3), J7.7 (Pin_7)
- net GLV-: now reaches U18. (GND_Lug)
- net at U16. (Tap3): now also K2.7, K2.8; no longer U18. (GND_Lug)
- net SDC2 renamed SDC5
- new net: U16. (Tap3), U18. (GND_Lug) (x4)
- no-connect marks 39 -> 44
Other:
- moved on the sheet: F10, R6
Changed lines of the file:
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@@
 	)
 	(junction
-		(at 45.085 126.365)
+		(at 45.72 126.365)
 		(diameter 0)
 		(color 255 153 0 1)
@@
 	)
 	(junction
-		(at 40.64 156.21)
-		(diameter 0)
-		(color 255 153 0 1)
-	)
-	(junction
 		(at 148.59 123.825)
 		(diameter 0)
@@
 	)
 	(junction
-		(at 50.165 156.21)
-		(diameter 0)
-		(color 255 153 0 1)
-	)
-	(junction
 		(at 67.31 156.21)
 		(diameter 0)
@@
 	)
 	(junction
+		(at 50.8 156.21)
+		(diameter 0)
+		(color 255 153 0 1)
+	)
+	(junction
+		(at 45.72 156.21)
+		(diameter 0)
+		(color 255 153 0 1)
+	)
+	(junction
 		(at 100.33 203.2)
 		(diameter 0)
@@
 	)
 	(junction
-		(at 45.085 156.21)
+		(at 41.91 156.21)
 		(diameter 0)
 		(color 255 153 0 1)
@@
 	)
 	(no_connect
+		(at 45.72 102.87)
+	)
+	(no_connect
 		(at 176.53 105.41)
 	)
@@
 	)
 	(no_connect
+		(at 41.91 102.87)
+	)
+	(no_connect
 		(at 220.98 200.66)
 	)
@@
 	)
 	(no_connect
+		(at 50.8 102.87)
+	)
+	(no_connect
 		(at 101.6 68.58)
 	)
@@
 	)
 	(no_connect
+		(at 100.33 102.87)
+	)
+	(no_connect
+		(at 48.26 102.87)
+	)
+	(no_connect
 		(at 217.17 264.16)
 	)
@@
 	(wire
 		(pts
-			(xy 47.625 126.365) (xy 45.085 126.365)
+			(xy 48.26 126.365) (xy 45.72 126.365)
 		)
 		(stroke
@@
 	(wire
 		(pts
-			(xy 45.085 156.21) (xy 40.64 156.21)
+			(xy 45.72 156.21) (xy 41.91 156.21)
 		)
 		(stroke
@@
 		)
 	)
-	(polyline
-		(pts
-			(xy 140.97 132.08) (xy 143.51 132.08)
-		)
-		(stroke
-			(width 0.254)
-			(type solid)
-			(color 0 0 132 1)
-		)
-	)
 	(wire
 		(pts
@@
 		)
 	)
-	(bus
-		(pts
-			(xy 227.33 210.82) (xy 227.33 208.28)
-		)
-		(stroke
-			(width 0)
-			(type default)
-		)
-	)
 	(wire
 		(pts
@@
 	(wire
 		(pts
-			(xy 45.085 128.905) (xy 45.085 126.365)
+			(xy 45.72 128.905) (xy 45.72 126.365)
 		)
 		(stroke
@@
 	(wire
 		(pts
-			(xy 40.64 129.54) (xy 40.64 102.87)
+			(xy 41.91 129.54) (xy 41.91 102.87)
 		)
 		(stroke
@@
 	(wire
 		(pts
-			(xy 45.085 126.365) (xy 45.085 102.87)
+			(xy 45.72 126.365) (xy 45.72 102.87)
 		)
 		(stroke
@@
 	(wire
 		(pts
-			(xy 45.085 156.21) (xy 45.085 136.525)
+			(xy 45.72 156.21) (xy 45.72 136.525)
 		)
 		(stroke
@@
 	(wire
 		(pts
-			(xy 57.15 156.21) (xy 50.165 156.21)
+			(xy 57.15 156.21) (xy 50.8 156.21)
 		)
 		(stroke
@@
 	(wire
 		(pts
-			(xy 50.165 156.21) (xy 45.085 156.21)
+			(xy 50.8 156.21) (xy 45.72 156.21)
 		)
 		(stroke
@@
 		)
 	)
+	(bus
+		(pts
+			(xy 140.97 132.08) (xy 143.51 132.08)
+		)
+		(stroke
+			(width 0)
+			(type default)
+		)
+	)
 	(wire
 		(pts
@@
 		)
 	)
+	(bus
+		(pts
+			(xy 227.33 147.32) (xy 227.33 210.82)
+		)
+		(stroke
+			(width 0)
+			(type default)
+		)
+	)
 	(wire
 		(pts
@@
 	(wire
 		(pts
-			(xy 50.165 156.21) (xy 50.165 102.87)
+			(xy 50.8 156.21) (xy 50.8 102.87)
 		)
 		(stroke
@@
 	(wire
 		(pts
-			(xy 47.625 126.365) (xy 47.625 102.87)
+			(xy 48.26 126.365) (xy 48.26 102.87)
 		)
 		(stroke
@@
 	(wire
 		(pts
-			(xy 40.64 156.21) (xy 40.64 137.16)
+			(xy 41.91 156.21) (xy 41.91 137.16)
 		)
 		(stroke
@@
 		)
 	)
-	(bus
-		(pts
-			(xy 227.33 208.28) (xy 227.33 205.74)
-		)
-		(stroke
-			(width 0)
-			(type default)
-		)
-	)
 	(wire
 		(pts
@@
 		)
 	)
-	(bus
+	(wire
 		(pts
-			(xy 140.97 146.05) (xy 227.33 146.05)
+			(xy 67.31 203.2) (xy 100.33 203.2)
 		)
 		(stroke
-			(width 0)
+			(width 0.508)
 			(type default)
+			(color 255 153 0 1)
 		)
 	)
-	(wire
+	(bus
 		(pts
-			(xy 67.31 203.2) (xy 100.33 203.2)
+			(xy 227.33 147.32) (xy 140.97 147.32)
 		)
 		(stroke
-			(width 0.508)
+			(width 0)
 			(type default)
-			(color 255 153 0 1)
 		)
 	)
@@
 		)
 	)
-	(bus
-		(pts
-			(xy 140.97 132.08) (xy 140.97 146.05)
-		)
-		(stroke
-			(width 0)
-			(type default)
-		)
-	)
 	(wire
 		(pts
@@
 	(wire
 		(pts
-			(xy 40.64 156.21) (xy 34.29 156.21)
+			(xy 34.29 156.21) (xy 41.91 156.21)
 		)
 		(stroke
@@
 		)
 	)
+	(bus
+		(pts
+			(xy 140.97 147.32) (xy 140.97 132.08)
+		)
+		(stroke
+			(width 0)
+			(type default)
+		)
+	)
 	(wire
 		(pts
@@
 		)
 	)
-	(bus
-		(pts
-			(xy 227.33 205.74) (xy 227.33 146.05)
-		)
-		(stroke
-			(width 0)
-			(type default)
-		)
-	)
 	(wire
 		(pts
@@
 		)
 	)
-	(label "SDC1"
+	(label "SDC4"
 		(at 147.32 109.22 270)
 		(effects
@@
 		)
 	)
-	(global_label "SDC2"
+	(global_label "SDC5"
 		(shape bidirectional)
 		(at 111.76 200.66 0)
@@
 		)
 	)
-	(global_label "SDC1"
+	(global_label "SDC4"
 		(shape input)
 		(at 121.92 107.95 270)
@@
 		)
 	)
-	(global_label "SDC2"
+	(global_label "SDC5"
 		(shape bidirectional)
 		(at 77.47 181.61 0)
@@
 		)
 	)
-	(global_label "SDC2"
+	(global_label "SDC5"
 		(shape bidirectional)
 		(at 85.725 271.907 0)
@@
 		)
 	)
-	(global_label "SDC1"
+	(global_label "SDC4"
 		(shape output)
 		(at 147.32 119.38 270)
@@
 		)
 	)
-	(global_label "SDC2"
+	(global_label "SDC5"
 		(shape output)
 		(at 120.65 107.95 270)
@@
 		)
 	)
-	(global_label "SDC2"
+	(global_label "SDC5"
 		(shape bidirectional)
 		(at 140.97 173.99 0)
@@
 	(symbol
 		(lib_id "Device:Fuse")
-		(at 45.085 132.715 180)
+		(at 45.72 132.715 180)
 		(unit 1)
 		(body_style 1)
@@
 		(dnp no)
 		(property "Reference" "F10"
-			(at 46.99 133.9851 0)
+			(at 47.625 133.9851 0)
 			(show_name no)
 			(do_not_autoplace no)
@@
 		)
 		(property "Value" "Fuse"
-			(at 46.99 131.4451 0)
+			(at 47.625 131.4451 0)
 			(show_name no)
 			(do_not_autoplace no)
@@
 		)
 		(property "Footprint" ""
-			(at 46.863 132.715 90)
+			(at 47.498 132.715 90)
 			(hide yes)
 			(show_name no)
@@
 		)
 		(property "Datasheet" ""
-			(at 45.085 132.715 0)
+			(at 45.72 132.715 0)
 			(hide yes)
 			(show_name no)
@@
 		)
 		(property "Description" "Fuse"
-			(at 45.085 132.715 0)
+			(at 45.72 132.715 0)
 			(hide yes)
 			(show_name no)
@@
 		(dnp no)
 		(property "Reference" "J20"
-			(at 162.306 209.55 0)
+			(at 162.56 209.042 0)
 			(show_name no)
 			(do_not_autoplace no)
@@
 			)
 		)
-		(property "Value" "GND"
+		(property "Value" "GLV-"
 			(at 79.375 251.587 0)
 			(show_name no)
@@
 	(symbol
 		(lib_id "Device:R_US")
-		(at 40.64 133.35 0)
+		(at 41.91 133.35 0)
 		(unit 1)
 		(body_style 1)
@@
 		(dnp no)
 		(property "Reference" "R6"
-			(at 38.1 133.35 90)
+			(at 39.37 133.35 90)
 			(show_name no)
 			(do_not_autoplace no)
@@
 		)
 		(property "Value" "RCH50S15001JS06"
-			(at 36.195 133.35 90)
+			(at 37.465 133.35 90)
 			(show_name no)
 			(do_not_autoplace no)
@@
 		)
 		(property "Footprint" ""
-			(at 41.656 133.604 90)
+			(at 42.926 133.604 90)
 			(hide yes)
 			(show_name no)
@@
 		)
 		(property "Datasheet" ""
-			(at 40.64 133.35 0)
+			(at 41.91 133.35 0)
 			(hide yes)
 			(show_name no)
@@
 		)
 		(property "Description" ""
-			(at 40.64 133.35 0)
+			(at 41.91 133.35 0)
 			(hide yes)
 			(show_name no)

Commit message: aesthetic changes
Connections:
- net at U16. (Tap3): now also K2.7, K2.8; no longer U18. (GND_Lug)
- new net: U16. (Tap3), U18. (GND_Lug) (x4)
Other:
- company: (none) -> SCFE27
- title: (none) -> Charge Cart + Tractive Battery
Changed lines of the file:
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@@
 	(generator_version "10.0")
 	(paper "A3")
+	(title_block
+		(title "Charge Cart + Tractive Battery")
+		(date "2026-10-27")
+		(rev "A")
+		(company "SCFE27")
+	)
 	(rectangle
 		(start 117.602 98.298)

Commit message: aesthetic changes
Connections:
- net at U16. (Tap3): now also K2.7, K2.8; no longer U18. (GND_Lug)
- new net: U16. (Tap3), U18. (GND_Lug) (x4)
Changed lines of the file:
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@@
 	(generator "eeschema")
 	(generator_version "10.0")
-	(paper "A3")
+	(paper "A3" portrait)
 	(title_block
 		(title "Charge Cart + Tractive Battery")

Commit message: chargecart + hvbp completed
Parts:
- added J10, J12, J9: DTM06-12SA, symbol Connector:Conn_01x12_Pin
- added J6, J8: UPCP012ALS2, symbol Connector:Conn_01x04_Pin
Connections:
- net CANGND_BMS is gone; now on net CANH: J7.10 (Pin_10)
- net CANH_BMS is gone; now on net CANL: J7.9 (Pin_9)
- net CANL_BMS is gone; now on net CANS: J7.8 (Pin_8)
- net IMD_fault is gone; now on net IMD_Fault: J7.12 (Pin_12), U12.8 (OKHS)
- net BMS_Fault: now also J7.1 (Pin_1), U18.7 (DES), J10.1 (Pin_1), J9.11 (Pin_11)
- net CANH: now also J10.10 (Pin_10), J9.10 (Pin_10)
- net CANL: now also J10.9 (Pin_9), J9.9 (Pin_9)
- net CANS: now also J10.8 (Pin_8), J9.8 (Pin_8)
- net CSS: now also J13.10 (Pin_10), J12.10 (Pin_10), J9.3 (Pin_3); no longer J13.4 (Pin_4)
- net GLV+: now also J10.6 (Pin_6), J9.6 (Pin_6)
- net GLV-: now also J13.11 (Pin_11), J13.9 (Pin_9), U18.29 (GND_Lug), J12.11 (Pin_11), J12.9 (Pin_9), J9.4 (Pin_4), J9.5 (Pin_5); no longer J13.3 (Pin_3), U18. (GND_Lug)
- net HV+_preres: now also U6.9 (HV+_preair); no longer U6. (HV-_postair)
- net IMD_Fault: now also J10.12 (Pin_12), J9.12 (Pin_12)
- net PostAIR+: now also U5.3 (HV+), U6.11 (HV+_postair); no longer U5. (HV-), U6. (HV-_postair)
- net PostAIR-: now also U5.4 (HV-), U6.10 (HV-_preair), U6.12 (HV-_postair); no longer U5. (HV-), U6. (HV-_postair)
- net SDC4: now also J10.7 (Pin_7), J9.7 (Pin_7)
- net at D3.1 (K): now also U5.2 (LED-); no longer U5. (HV-)
- net at D3.2 (A): now also U5.1 (LED+); no longer U5. (HV-)
- net at F2.1: now also U16.1 (HV-); no longer U16. (Tap3)
- net at U4.DC1 (HV+): now also F5.1, J1.3 (Pin_2); no longer F3.1
- net at K2.7, K2.8: now also U16.1 (HV-); no longer U16. (Tap3)
- net BMS_fault: no longer names the net of J7.11 (Pin_11)
- net BMS_fault: no longer U18.7 (DES)
- new net: U16.3 (Therm), U18.25 (Therm)
- new net: U16.4 (Tap1), U18.26 (Tap1)
- new net: U16.5 (Tap2), U18.27 (Tap2)
- new net: U16.6 (Tap3), U18.28 (Tap3)
- new net: J6.1 (Pin_1), J6.2 (Pin_2)
- new net: J6.3 (Pin_3), J8.3 (Pin_3)
- new net: J6.4 (Pin_4), J8.4 (Pin_4)
- new net: F3.1, U4.DC2 (HV-)
- new net: J8.1 (Pin_1), J8.2 (Pin_2)
- no-connect marks 44 -> 59
Other:
- note added: "External Harnesses"
- note added: "HV (Charge Cart)"
- note added: "LV (Acc Chg)"
- note added: "LV (Acc Chk)"
- note added: "LV (Charge Cart)"
- note added: "LV Harness (Chg)"
- note added: "LV Harness (Chk)"
- note added: "Wire Gauges"
- note added: "dark orange: 10awg [ charge cart internal HV DC ]"
- note added: "green: 22awg [ LV ]"
- note added: "magenta: 10awg [ charge cart internal HV AC ]"
- note added: "orange: 20awg [ HV sense: TSMP, IMD, indicator, precharge ]"
- note added: "orange: 4awg [ accumulator internal HV ]"
- note added: "red: 4awg shielded [ external HV harness ]"
- note removed: "32A fuses"
