File: 2026-27/Boards/ariczhan_VIL_RML_full_sim/integrated_vil_rml.kicad_pcb (KiCad board)
At the start: 2 copper layers, 90.1 x 30 mm, 31 parts, among them J1 043045-0412, Q2 AO3400A, Q3 UJ3N065080K3S, Q4 AO3401A, U1 H11L1, U2 NE555

Commit message: fixed integrated vil rml final fr fr this time
Connections:
- Molex1 pad 2: unconnected-(Molex1-Pin_2-Pad2) -> /HV+
- Molex2 pad 2: unconnected-(Molex2-Pin_2-Pad2) -> Net-(Molex2-Pin_1)
Routing:
- net Net-(Molex2-Pin_1): track 10.6 -> 13.6 mm
- net /HV+: track 5.22 -> 8.22 mm
- net Net-(D3-A): vias 0 -> 118
- added copper zone on B.Cu, net Net-(D3-A)
- added copper zone on F.Cu, net Net-(D3-A)
